File: backbone/backbone.kicad_pcb (KiCad board)
At the start: 4 copper layers, 0 parts

Commit message: before hand editing
Parts:
- added C1001: 100nF, 0_backbone:C_0603, F.Cu at (141.9, 107.9)
- added C1002: 10uF, 0_backbone:C_0805, F.Cu at (159.7, 103.5)
- added C1003: 47uF 10V, 0_backbone:C_1206, F.Cu at (148.6, 103.7)
- added C1004: 100nF, 0_backbone:C_0603, F.Cu at (146.0, 107.9)
- added C1005: 100nF, 0_backbone:C_0402, F.Cu at (161.1, 107.7)
- added C1006: 100nF, 0_backbone:C_0402, F.Cu at (164.1, 107.7)
- added C1007: 1nF 2kV, 0_backbone:C_1206, F.Cu at (154.5, 103.7)
- added C1101: 33pF, 0_backbone:C_0603, F.Cu at (53.7, 62.1)
- added C1102: 33pF, 0_backbone:C_0603, F.Cu at (57.7, 62.1)
- added C1103: 100nF, 0_backbone:C_0603, F.Cu at (61.8, 62.1)
- added C1104: 100nF, 0_backbone:C_0603, F.Cu at (65.8, 62.1)
- added C1105: 100nF, 0_backbone:C_0603, F.Cu at (69.9, 62.1)
- added C1106: 100nF, 0_backbone:C_0603, F.Cu at (73.9, 62.1)
- added C1107: 100nF, 0_backbone:C_0603, F.Cu at (78.0, 62.1)
- added C1108: 10uF, 0_backbone:C_0805, F.Cu at (78.1, 47.5)
- added C1201: 100nF, 0_backbone:C_0603, F.Cu at (15.2, 109.3)
- added C1202: 100nF, 0_backbone:C_0603, F.Cu at (19.2, 109.3)
- added C1203: 100nF, 0_backbone:C_0603, F.Cu at (23.3, 109.3)
- added C1204: 100nF, 0_backbone:C_0603, F.Cu at (27.3, 109.3)
- added C1205: 470uF 25V, 0_backbone:CAP-SMD_BD8.0-L8.3-W8.3-LS9.0-FD_H10.5, F.Cu at (7.61, 84.8)
- added C1206: 100nF, 0_backbone:C_0603, F.Cu at (3.92, 113.0)
- added C1207: 100nF, 0_backbone:C_0603, F.Cu at (7.97, 113.0)
- added C1208: 470uF 10V, 0_backbone:CAP-SMD_BD6.3-L6.6-W6.6-LS7.3-FD-H7.7, F.Cu at (18.3, 84.0)
- added C1209: 100nF, 0_backbone:C_0603, F.Cu at (12.0, 113.0)
- added C1301: 100nF, 0_backbone:C_0603, F.Cu at (48.7, 109.3)
- added C1302: 100nF, 0_backbone:C_0603, F.Cu at (52.7, 109.3)
- added C1303: 100nF, 0_backbone:C_0603, F.Cu at (56.8, 109.3)
- added C1304: 100nF, 0_backbone:C_0603, F.Cu at (60.8, 109.3)
- added C1305: 470uF 25V, 0_backbone:CAP-SMD_BD8.0-L8.3-W8.3-LS9.0-FD_H10.5, F.Cu at (41.1, 84.8)
- added C1306: 100nF, 0_backbone:C_0603, F.Cu at (37.4, 113.0)
- added C1307: 100nF, 0_backbone:C_0603, F.Cu at (41.5, 113.0)
- added C1308: 470uF 10V, 0_backbone:CAP-SMD_BD6.3-L6.6-W6.6-LS7.3-FD-H7.7, F.Cu at (51.8, 84.0)
- added C1309: 100nF, 0_backbone:C_0603, F.Cu at (45.5, 113.0)
- added C1401: 100nF, 0_backbone:C_0603, F.Cu at (82.2, 109.3)
- added C1402: 100nF, 0_backbone:C_0603, F.Cu at (86.2, 109.3)
- added C1403: 100nF, 0_backbone:C_0603, F.Cu at (90.3, 109.3)
- added C1404: 100nF, 0_backbone:C_0603, F.Cu at (94.3, 109.3)
- added C1405: 470uF 25V, 0_backbone:CAP-SMD_BD8.0-L8.3-W8.3-LS9.0-FD_H10.5, F.Cu at (74.6, 84.8)
- added C1406: 100nF, 0_backbone:C_0603, F.Cu at (70.9, 113.0)
- added C1407: 100nF, 0_backbone:C_0603, F.Cu at (75.0, 113.0)
- added C1408: 470uF 10V, 0_backbone:CAP-SMD_BD6.3-L6.6-W6.6-LS7.3-FD-H7.7, F.Cu at (85.3, 84.0)
- added C1409: 100nF, 0_backbone:C_0603, F.Cu at (79.0, 113.0)
- added C1501: 100nF, 0_backbone:C_0603, F.Cu at (115.7, 109.3)
- added C1502: 100nF, 0_backbone:C_0603, F.Cu at (119.7, 109.3)
- added C1503: 100nF, 0_backbone:C_0603, F.Cu at (123.8, 109.3)
- added C1504: 100nF, 0_backbone:C_0603, F.Cu at (127.8, 109.3)
- added C1505: 470uF 25V, 0_backbone:CAP-SMD_BD8.0-L8.3-W8.3-LS9.0-FD_H10.5, F.Cu at (108.1, 84.8)
- added C1506: 100nF, 0_backbone:C_0603, F.Cu at (104.4, 113.0)
- added C1507: 100nF, 0_backbone:C_0603, F.Cu at (108.5, 113.0)
- added C1508: 470uF 10V, 0_backbone:CAP-SMD_BD6.3-L6.6-W6.6-LS7.3-FD-H7.7, F.Cu at (118.8, 84.0)
- added C1509: 100nF, 0_backbone:C_0603, F.Cu at (112.5, 113.0)
- added C201: 100nF, 0_backbone:C_0603, F.Cu at (31.8, 36.0)
- added C202: 470uF 35V, 0_backbone:CAP-SMD_BD10.0-L10.3-W10.3-LS11.3-FD, F.Cu at (25.0, 7.80)
- added C203: 470uF 35V, 0_backbone:CAP-SMD_BD10.0-L10.3-W10.3-LS11.3-FD, F.Cu at (25.0, 19.6)
- added C204: 10uF 50V, 0_backbone:C_1206, F.Cu at (26.4, 33.0)
- added C205: 100nF 100V, 0_backbone:C_0805, F.Cu at (19.9, 36.4)
- added C206: 10uF 50V, 0_backbone:C_1206, F.Cu at (32.3, 33.0)
- added C301: 33nF, 0_backbone:C_0603, F.Cu at (72.6, 29.9)
- added C302: 3.3nF, 0_backbone:C_0603, F.Cu at (76.6, 29.9)
- added C303: 47pF, 0_backbone:C_0603, F.Cu at (80.7, 29.9)
- added C304: 680pF, 0_backbone:C_0603, F.Cu at (84.7, 29.9)
- added C305: 2.2uF, 0_backbone:C_0603, F.Cu at (88.8, 29.9)
- added C306: 100nF, 0_backbone:C_0603, F.Cu at (92.8, 29.9)
- added C307: 100nF 100V, 0_backbone:C_0805, F.Cu at (60.7, 30.3)
- added C308: 10pF, 0_backbone:C_0603, F.Cu at (49.9, 33.9)
- added C309: 4.7uF 100V, 0_backbone:C1210, F.Cu at (73.4, 18.2)
- added C310: 4.7uF 100V, 0_backbone:C1210, F.Cu at (79.8, 18.2)
- added C311: 4.7uF 100V, 0_backbone:C1210, F.Cu at (86.3, 18.2)
- added C312: 4.7uF 100V, 0_backbone:C1210, F.Cu at (92.8, 18.2)
- added C313: 4.7uF 100V, 0_backbone:C1210, F.Cu at (51.1, 26.4)
- added C314: 47uF 16V, 0_backbone:C1210, F.Cu at (57.6, 26.4)
- added C315: 47uF 16V, 0_backbone:C1210, F.Cu at (64.1, 26.4)
- added C316: 47uF 16V, 0_backbone:C1210, F.Cu at (70.5, 26.4)
- added C317: 47uF 16V, 0_backbone:C1210, F.Cu at (77.0, 26.4)
- added C318: 22uF 25V, 0_backbone:C1210, F.Cu at (83.5, 26.4)
- added C319: 22uF 25V, 0_backbone:C1210, F.Cu at (90.0, 26.4)
- added C320: 470uF 25V, 0_backbone:CAP-SMD_BD8.0-L8.3-W8.3-LS9.0-FD_H10.5, F.Cu at (70.3, 6.80)
- added C321: 470uF 25V, 0_backbone:CAP-SMD_BD8.0-L8.3-W8.3-LS9.0-FD_H10.5, F.Cu at (81.7, 6.80)
- added C322: 100pF, 0_backbone:C_0603, F.Cu at (54.0, 33.9)
- added C401: 47nF, 0_backbone:C_0603, F.Cu at (118.7, 26.8)
- added C402: 4.7nF, 0_backbone:C_0603, F.Cu at (122.8, 26.8)
- added C403: 150pF, 0_backbone:C_0603, F.Cu at (126.8, 26.8)
- added C404: 1.8nF, 0_backbone:C_0603, F.Cu at (130.9, 26.8)
- added C405: 2.2uF, 0_backbone:C_0603, F.Cu at (134.9, 26.8)
- added C406: 100nF, 0_backbone:C_0603, F.Cu at (139.0, 26.8)
- added C407: 100nF 100V, 0_backbone:C_0805, F.Cu at (106.9, 27.2)
- added C408: 15pF, 0_backbone:C_0603, F.Cu at (101.9, 30.5)
- added C409: 2.2uF 100V, 0_backbone:C1210, F.Cu at (110.2, 18.2)
- added C410: 2.2uF 100V, 0_backbone:C1210, F.Cu at (116.7, 18.2)
- added C411: 2.2uF 100V, 0_backbone:C1210, F.Cu at (123.1, 18.2)
- added C412: 2.2uF 100V, 0_backbone:C1210, F.Cu at (129.6, 18.2)
- added C413: 2.2uF 100V, 0_backbone:C1210, F.Cu at (136.1, 18.2)
- added C414: 47uF 10V, 0_backbone:C_1206, F.Cu at (108.7, 23.3)
- added C415: 47uF 10V, 0_backbone:C_1206, F.Cu at (114.5, 23.3)
- added C416: 47uF 10V, 0_backbone:C_1206, F.Cu at (120.4, 23.3)
- added C417: 47uF 10V, 0_backbone:C_1206, F.Cu at (126.2, 23.3)
- added C418: 47uF 10V, 0_backbone:C_1206, F.Cu at (132.1, 23.3)
- added C419: 47uF 10V, 0_backbone:C_1206, F.Cu at (137.9, 23.3)
- added C420: 470uF 10V, 0_backbone:CAP-SMD_BD6.3-L6.6-W6.6-LS7.3-FD-H7.7, F.Cu at (120.6, 5.96)
- added C421: 100pF, 0_backbone:C_0603, F.Cu at (106.0, 30.5)
- added C501: 4.7nF, 0_backbone:C_0603, F.Cu at (157.4, 25.2)
- added C502: 47pF, 0_backbone:C_0603, F.Cu at (161.5, 25.2)
- added C503: 100nF, 0_backbone:C_0603, F.Cu at (165.5, 25.2)
- added C504: 2.2uF 100V, 0_backbone:C1210, F.Cu at (157.4, 15.8)
- added C505: 2.2uF 100V, 0_backbone:C1210, F.Cu at (163.9, 15.8)
- added C506: 2.2uF 100V, 0_backbone:C1210, F.Cu at (170.4, 15.8)
- added C507: 2.2uF 100V, 0_backbone:C1210, F.Cu at (176.8, 15.8)
- added C508: 47uF 16V, 0_backbone:C1210, F.Cu at (183.3, 15.8)
- added C509: 47uF 16V, 0_backbone:C1210, F.Cu at (151.1, 21.8)
- added C510: 47uF 16V, 0_backbone:C1210, F.Cu at (157.6, 21.8)
- added C511: 6.8pF, 0_backbone:C_0603, F.Cu at (169.6, 25.2)
- added C512: 4.7uF, 0_backbone:C_0805, F.Cu at (177.4, 21.1)
- added C513: 22uF, 0_backbone:C_0805, F.Cu at (182.1, 21.1)
- added C601: 100nF, 0_backbone:C_0402, F.Cu at (153.0, 51.5)
- added C602: 100nF, 0_backbone:C_0402, F.Cu at (156.1, 51.5)
- added C603: 100nF, 0_backbone:C_0603, F.Cu at (166.5, 47.1)
- added C604: 100nF, 0_backbone:C_0603, F.Cu at (170.6, 47.1)
- added C605: 1uF, 0_backbone:C_0603, F.Cu at (174.6, 47.1)
- added C606: 100nF, 0_backbone:C_0603, F.Cu at (137.9, 51.7)
- added C607: 1nF 2kV, 0_backbone:C_1206, F.Cu at (149.8, 47.7)
- added C701: 10uF, 0_backbone:C_0805, F.Cu at (121.6, 47.5)
- added C702: 30pF, 0_backbone:C_0603, F.Cu at (119.6, 58.7)
- added C703: 30pF, 0_backbone:C_0603, F.Cu at (123.6, 58.7)
- added C704: 6.8pF, 0_backbone:C_0603, F.Cu at (127.7, 58.7)
- added C705: 4.7uF, 0_backbone:C_0805, F.Cu at (126.2, 47.5)
- added C706: 22uF, 0_backbone:C_0805, F.Cu at (94.2, 59.1)
- added C707: 100nF, 0_backbone:C_0603, F.Cu at (93.9, 62.4)
- added C708: 100nF, 0_backbone:C_0603, F.Cu at (98.0, 62.4)
- added C709: 100nF, 0_backbone:C_0603, F.Cu at (102.0, 62.4)
- added C710: 100nF, 0_backbone:C_0603, F.Cu at (106.1, 62.4)
- added C711: 100nF, 0_backbone:C_0603, F.Cu at (110.1, 62.4)
- added C712: 100nF, 0_backbone:C_0603, F.Cu at (114.2, 62.4)
- added C713: 100nF, 0_backbone:C_0603, F.Cu at (118.2, 62.4)
- added C714: 100nF, 0_backbone:C_0603, F.Cu at (122.3, 62.4)
- added C715: 10uF, 0_backbone:C_0805, F.Cu at (98.9, 59.1)
- added C716: 100nF, 0_backbone:C_0603, F.Cu at (126.3, 62.4)
- added C717: 100nF, 0_backbone:C_0603, F.Cu at (93.9, 64.9)
- added C718: 100nF, 0_backbone:C_0603, F.Cu at (98.0, 64.9)
- added C719: 100nF, 0_backbone:C_0603, F.Cu at (102.0, 64.9)
- added C720: 10uF, 0_backbone:C_0805, F.Cu at (103.5, 59.1)
- added C801: 100nF, 0_backbone:C_0603, F.Cu at (141.9, 73.9)
- added C802: 10uF, 0_backbone:C_0805, F.Cu at (159.7, 69.5)
- added C803: 47uF 10V, 0_backbone:C_1206, F.Cu at (148.6, 69.7)
- added C804: 100nF, 0_backbone:C_0603, F.Cu at (146.0, 73.9)
- added C805: 100nF, 0_backbone:C_0402, F.Cu at (161.1, 73.7)
- added C806: 100nF, 0_backbone:C_0402, F.Cu at (164.1, 73.7)
- added C807: 1nF 2kV, 0_backbone:C_1206, F.Cu at (154.5, 69.7)
- added C901: 100nF, 0_backbone:C_0603, F.Cu at (141.9, 90.9)
- added C902: 10uF, 0_backbone:C_0805, F.Cu at (159.7, 86.5)
- added C903: 47uF 10V, 0_backbone:C_1206, F.Cu at (148.6, 86.7)
- added C904: 100nF, 0_backbone:C_0603, F.Cu at (146.0, 90.9)
- added C905: 100nF, 0_backbone:C_0402, F.Cu at (161.1, 90.7)
- added C906: 100nF, 0_backbone:C_0402, F.Cu at (164.1, 90.7)
- added C907: 1nF 2kV, 0_backbone:C_1206, F.Cu at (154.5, 86.7)
- added D1001: USBLC6-2SC6, 0_backbone:SOT-23-6_L2.9-W1.6-P0.95-LS2.8-BL, F.Cu at (143.5, 104.2)
- added D1002: TPD4E05U06, 0_backbone:USON-10_L2.5-W1.0-P0.50-BL, F.Cu at (137.9, 108.0)
- added D1101: LED ACT, 0_backbone:D_0805, F.Cu at (73.5, 47.5)
- added D1102: USBLC6-2SC6, 0_backbone:SOT-23-6_L2.9-W1.6-P0.95-LS2.8-BL, F.Cu at (68.9, 48.2)
- added D1201: PSM712-LF-T7, 0_backbone:SOT-23-3_L3.0-W1.7-P0.95-LS2.9-BR, F.Cu at (18.6, 100.5)
- added D1202: SMF5.0A, 0_backbone:D_SOD-123FL, F.Cu at (23.9, 100.1)
- added D1203: SMBJ13A, 0_backbone:D_SMB, F.Cu at (21.3, 92.6)
- added D1204: SMBJ6.0A, 0_backbone:D_SMB, F.Cu at (6.24, 101.2)
- added D1301: PSM712-LF-T7, 0_backbone:SOT-23-3_L3.0-W1.7-P0.95-LS2.9-BR, F.Cu at (52.1, 100.5)
- added D1302: SMF5.0A, 0_backbone:D_SOD-123FL, F.Cu at (57.4, 100.1)
- added D1303: SMBJ13A, 0_backbone:D_SMB, F.Cu at (54.8, 92.6)
- added D1304: SMBJ6.0A, 0_backbone:D_SMB, F.Cu at (39.7, 101.2)
- added D1401: PSM712-LF-T7, 0_backbone:SOT-23-3_L3.0-W1.7-P0.95-LS2.9-BR, F.Cu at (85.6, 100.5)
- added D1402: SMF5.0A, 0_backbone:D_SOD-123FL, F.Cu at (90.9, 100.1)
- added D1403: SMBJ13A, 0_backbone:D_SMB, F.Cu at (88.3, 92.6)
- added D1404: SMBJ6.0A, 0_backbone:D_SMB, F.Cu at (73.2, 101.2)
- added D1501: PSM712-LF-T7, 0_backbone:SOT-23-3_L3.0-W1.7-P0.95-LS2.9-BR, F.Cu at (119.1, 100.5)
- added D1502: SMF5.0A, 0_backbone:D_SOD-123FL, F.Cu at (124.4, 100.1)
- added D1503: SMBJ13A, 0_backbone:D_SMB, F.Cu at (121.8, 92.6)
- added D1504: SMBJ6.0A, 0_backbone:D_SMB, F.Cu at (106.7, 101.2)
- added D201: SMBJ24A, 0_backbone:D_SMB, F.Cu at (22.0, 28.4)
- added D202: LED Green, 0_backbone:D_0805, F.Cu at (37.6, 32.9)
- added D301: SS14, 0_backbone:D_SMA, F.Cu at (66.0, 18.3)
- added D302: LED Green, 0_backbone:D_0805, F.Cu at (56.1, 30.3)
- added D401: LED Green, 0_backbone:D_0805, F.Cu at (102.3, 27.2)
- added D501: B560C, 0_backbone:SMC_L7.1-W6.2-LS8.1-RD, F.Cu at (165.7, 5.73)
- added D502: LED Green, 0_backbone:D_0805, F.Cu at (168.1, 21.1)
- added D503: LED Green, 0_backbone:D_0805, F.Cu at (172.8, 21.1)
- added D601: TPD4E05U06, 0_backbone:USON-10_L2.5-W1.0-P0.50-BL, F.Cu at (158.5, 47.2)
- added D602: TPD4E05U06, 0_backbone:USON-10_L2.5-W1.0-P0.50-BL, F.Cu at (162.5, 47.2)
- added D603: USBLC6-2SC6, 0_backbone:SOT-23-6_L2.9-W1.6-P0.95-LS2.8-BL, F.Cu at (144.7, 48.2)
- added D801: USBLC6-2SC6, 0_backbone:SOT-23-6_L2.9-W1.6-P0.95-LS2.8-BL, F.Cu at (143.5, 70.2)
- added D802: TPD4E05U06, 0_backbone:USON-10_L2.5-W1.0-P0.50-BL, F.Cu at (137.9, 74.0)
- added D901: USBLC6-2SC6, 0_backbone:SOT-23-6_L2.9-W1.6-P0.95-LS2.8-BL, F.Cu at (143.5, 87.2)
- added D902: TPD4E05U06, 0_backbone:USON-10_L2.5-W1.0-P0.50-BL, F.Cu at (137.9, 91.0)
- added F201: 15A T 2410, 0_backbone:FUSE-SMD_L6.1-W2.7, F.Cu at (31.0, 28.0)
- added F202: 4A T 1206, 0_backbone:F1206, F.Cu at (20.6, 33.0)
- added FB1001: BLM21PG221SN1D, 0_backbone:FB_0805, F.Cu at (164.4, 103.4)
- added FB701: BLM18PG221SN1D, 0_backbone:FB_0603, F.Cu at (115.5, 58.8)
- added FB801: BLM21PG221SN1D, 0_backbone:FB_0805, F.Cu at (164.4, 69.4)
- added FB901: BLM21PG221SN1D, 0_backbone:FB_0805, F.Cu at (164.4, 86.4)
- added H101: M3, 0_backbone:MountingHole_3.2mm_M3_Pad_Via, F.Cu at (4.50, 4.50)
- added H102: M3, 0_backbone:MountingHole_3.2mm_M3_Pad_Via, F.Cu at (185.5, 4.50)
- added H103: M3, 0_backbone:MountingHole_3.2mm_M3_Pad_Via, F.Cu at (4.50, 125.5)
- added H104: M3, 0_backbone:MountingHole_3.2mm_M3_Pad_Via, F.Cu at (185.5, 125.5)
- added J1001: USB-A 3.0 receptacle, 0_backbone:USB-3.0-A-TH_HC-ST-003-01-Z, F.Cu at (183.6, 110.5)
- added J1201: RS-485 JST EH 4p, 0_backbone:CONN-TH_B4B-EH-A-LF-SN, F.Cu at (16.9, 124.6)
- added J1202: TTL JST EH 3p, 0_backbone:CONN-TH_B3B-EH-A-LF-SN, F.Cu at (29.7, 124.4)
- added J1301: RS-485 JST EH 4p, 0_backbone:CONN-TH_B4B-EH-A-LF-SN, F.Cu at (42.4, 124.6)
- added J1302: TTL JST EH 3p, 0_backbone:CONN-TH_B3B-EH-A-LF-SN, F.Cu at (55.2, 124.4)
- added J1401: RS-485 JST EH 4p, 0_backbone:CONN-TH_B4B-EH-A-LF-SN, F.Cu at (75.9, 124.6)
- added J1402: TTL JST EH 3p, 0_backbone:CONN-TH_B3B-EH-A-LF-SN, F.Cu at (88.7, 124.4)
- added J1501: RS-485 JST EH 4p, 0_backbone:CONN-TH_B4B-EH-A-LF-SN, F.Cu at (109.4, 124.6)
- added J1502: TTL JST EH 3p, 0_backbone:CONN-TH_B3B-EH-A-LF-SN, F.Cu at (122.2, 124.4)
- added J201: XT30PW-M, 0_backbone:CONN-TH_XT30PW-M, F.Cu at (9.35, 17.3)
- added J202: XT30PW-M, 0_backbone:CONN-TH_XT30PW-M, F.Cu at (9.35, 32.0)
- added J601: USB-C 24P receptacle, 0_backbone:USB-C-SMD_TYPE-C-24P-QT, F.Cu at (183.8, 51.4)
- added J801: USB-A 3.0 receptacle, 0_backbone:USB-3.0-A-TH_HC-ST-003-01-Z, F.Cu at (183.6, 76.5)
- added J901: USB-A 3.0 receptacle, 0_backbone:USB-3.0-A-TH_HC-ST-003-01-Z, F.Cu at (183.6, 93.5)
- added JP1201: MODE: 1-2 RS-485 (default), 2-3 TTL, 0_backbone:SolderJumper-3_P1.3mm_Bridged12_RoundedPad1.0x1.5mm, F.Cu at (13.4, 100.2)
- added JP1202: MODE: bridged = auto-retry, open = latch-off, 0_backbone:SolderJumper-2_P1.3mm_Bridged_RoundedPad1.0x1.5mm, F.Cu at (9.08, 105.9)
- added JP1301: MODE: 1-2 RS-485 (default), 2-3 TTL, 0_backbone:SolderJumper-3_P1.3mm_Bridged12_RoundedPad1.0x1.5mm, F.Cu at (46.9, 100.2)
- added JP1302: MODE: bridged = auto-retry, open = latch-off, 0_backbone:SolderJumper-2_P1.3mm_Bridged_RoundedPad1.0x1.5mm, F.Cu at (42.6, 105.9)
- added JP1401: MODE: 1-2 RS-485 (default), 2-3 TTL, 0_backbone:SolderJumper-3_P1.3mm_Bridged12_RoundedPad1.0x1.5mm, F.Cu at (80.4, 100.2)
- added JP1402: MODE: bridged = auto-retry, open = latch-off, 0_backbone:SolderJumper-2_P1.3mm_Bridged_RoundedPad1.0x1.5mm, F.Cu at (76.1, 105.9)
- added JP1501: MODE: 1-2 RS-485 (default), 2-3 TTL, 0_backbone:SolderJumper-3_P1.3mm_Bridged12_RoundedPad1.0x1.5mm, F.Cu at (113.9, 100.2)
- added JP1502: MODE: bridged = auto-retry, open = latch-off, 0_backbone:SolderJumper-2_P1.3mm_Bridged_RoundedPad1.0x1.5mm, F.Cu at (109.6, 105.9)
- added JP301: SYNCIN: 1-2 GND=DEM, 2-3 VCC=FPWM, 0_backbone:SolderJumper-3_P1.3mm_Bridged12_RoundedPad1.0x1.5mm, F.Cu at (50.8, 30.5)
- added JP401: SYNCIN: 1-2 GND=DEM, 2-3 VCC=FPWM, 0_backbone:SolderJumper-3_P1.3mm_Bridged12_RoundedPad1.0x1.5mm, F.Cu at (102.8, 23.4)
- added L301: 4.7uH 20A, 0_backbone:IND-SMD_L13.5-W12.6, F.Cu at (56.2, 8.93)
- added L401: 3.3uH 18A, 0_backbone:IND-SMD_L13.5-W12.6_125CDMCC-DS, F.Cu at (107.8, 8.88)
- added L501: 7.2uH 6A, 0_backbone:IND-SMD_L10.2-W10.2_7447798720, F.Cu at (154.1, 7.72)
- added L502: 2.2uH 3.4A, 0_backbone:IND-SMD_L4.0-W4.0_LQH44PN2R2MP0L, F.Cu at (151.1, 16.5)
- added L701: 2.2uH 3.4A, 0_backbone:IND-SMD_L4.0-W4.0_LQH44PN2R2MP0L, F.Cu at (105.9, 48.9)
- added Q201: CSD18532Q5B, 0_backbone:SON-8_L5.0-W6.0-P1.27-BL-1, F.Cu at (35.8, 17.6)
- added Q301: CSD18532Q5B, 0_backbone:SON-8_L5.0-W6.0-P1.27-BL-1, F.Cu at (90.9, 5.80)
- added Q302: CSD18532Q5B, 0_backbone:SON-8_L5.0-W6.0-P1.27-BL-1, F.Cu at (51.3, 19.9)
- added Q401: CSD18532Q5B, 0_backbone:SON-8_L5.0-W6.0-P1.27-BL-1, F.Cu at (129.1, 5.80)
- added Q402: CSD18532Q5B, 0_backbone:SON-8_L5.0-W6.0-P1.27-BL-1, F.Cu at (136.0, 5.80)
- added R1001: 16.9k, 0_backbone:R_0603, F.Cu at (149.9, 107.9)
- added R1002: 10k, 0_backbone:R_0603, F.Cu at (153.8, 107.9)
- added R1003: 1M, 0_backbone:R_0603, F.Cu at (157.6, 107.9)
- added R1101: 10k, 0_backbone:R_0603, F.Cu at (81.9, 62.1)
- added R1102: 4.7k, 0_backbone:R_0603, F.Cu at (85.8, 62.1)
- added R1103: 4.7k, 0_backbone:R_0603, F.Cu at (49.8, 65.8)
- added R1104: 4.7k, 0_backbone:R_0603, F.Cu at (53.7, 65.8)
- added R1105: 4.7k, 0_backbone:R_0603, F.Cu at (57.5, 65.8)
- added R1106: 1k, 0_backbone:R_0603, F.Cu at (61.4, 65.8)
- added R1201: 100k, 0_backbone:R_0603, F.Cu at (16.0, 113.0)
- added R1202: 100k, 0_backbone:R_0603, F.Cu at (19.8, 113.0)
- added R1203: 10k, 0_backbone:R_0603, F.Cu at (23.7, 113.0)
- added R1204: 120, 0_backbone:R_0603, F.Cu at (27.5, 113.0)
- added R1205: 22, 0_backbone:R_0603, F.Cu at (3.83, 115.5)
- added R1206: 10k, 0_backbone:R_0603, F.Cu at (7.67, 115.5)
- added R1207: 249k, 0_backbone:R_0603, F.Cu at (11.5, 115.5)
- added R1208: 18.2k, 0_backbone:R_0603, F.Cu at (15.4, 115.5)
- added R1209: 20.5k, 0_backbone:R_0603, F.Cu at (19.2, 115.5)
- added R1210: 4.02k, 0_backbone:R_0603, F.Cu at (23.1, 115.5)
- added R1211: 100k, 0_backbone:R_0603, F.Cu at (26.9, 115.5)
- added R1212: 27k, 0_backbone:R_0603, F.Cu at (3.83, 117.9)
- added R1213: 100k, 0_backbone:R_0603, F.Cu at (7.67, 117.9)
- added R1301: 100k, 0_backbone:R_0603, F.Cu at (49.5, 113.0)
- added R1302: 100k, 0_backbone:R_0603, F.Cu at (53.3, 113.0)
- added R1303: 10k, 0_backbone:R_0603, F.Cu at (57.2, 113.0)
- added R1304: 120, 0_backbone:R_0603, F.Cu at (61.0, 113.0)
- added R1305: 22, 0_backbone:R_0603, F.Cu at (37.3, 115.5)
- added R1306: 10k, 0_backbone:R_0603, F.Cu at (41.2, 115.5)
- added R1307: 249k, 0_backbone:R_0603, F.Cu at (45.0, 115.5)
- added R1308: 18.2k, 0_backbone:R_0603, F.Cu at (48.9, 115.5)
- added R1309: 20.5k, 0_backbone:R_0603, F.Cu at (52.7, 115.5)
- added R1310: 4.02k, 0_backbone:R_0603, F.Cu at (56.6, 115.5)
- added R1311: 100k, 0_backbone:R_0603, F.Cu at (60.4, 115.5)
- added R1312: 27k, 0_backbone:R_0603, F.Cu at (37.3, 117.9)
- added R1313: 100k, 0_backbone:R_0603, F.Cu at (41.2, 117.9)
- added R1401: 100k, 0_backbone:R_0603, F.Cu at (83.0, 113.0)
- added R1402: 100k, 0_backbone:R_0603, F.Cu at (86.8, 113.0)
- added R1403: 10k, 0_backbone:R_0603, F.Cu at (90.7, 113.0)
- added R1404: 120, 0_backbone:R_0603, F.Cu at (94.5, 113.0)
- added R1405: 22, 0_backbone:R_0603, F.Cu at (70.8, 115.5)
- added R1406: 10k, 0_backbone:R_0603, F.Cu at (74.7, 115.5)
- added R1407: 249k, 0_backbone:R_0603, F.Cu at (78.5, 115.5)
- added R1408: 18.2k, 0_backbone:R_0603, F.Cu at (82.4, 115.5)
- added R1409: 20.5k, 0_backbone:R_0603, F.Cu at (86.2, 115.5)
- added R1410: 4.02k, 0_backbone:R_0603, F.Cu at (90.1, 115.5)
- added R1411: 100k, 0_backbone:R_0603, F.Cu at (93.9, 115.5)
- added R1412: 27k, 0_backbone:R_0603, F.Cu at (70.8, 117.9)
- added R1413: 100k, 0_backbone:R_0603, F.Cu at (74.7, 117.9)
- added R1501: 100k, 0_backbone:R_0603, F.Cu at (116.5, 113.0)
- added R1502: 100k, 0_backbone:R_0603, F.Cu at (120.3, 113.0)
- added R1503: 10k, 0_backbone:R_0603, F.Cu at (124.2, 113.0)
- added R1504: 120, 0_backbone:R_0603, F.Cu at (128.0, 113.0)
- added R1505: 22, 0_backbone:R_0603, F.Cu at (104.3, 115.5)
- added R1506: 10k, 0_backbone:R_0603, F.Cu at (108.2, 115.5)
- added R1507: 249k, 0_backbone:R_0603, F.Cu at (112.0, 115.5)
- added R1508: 18.2k, 0_backbone:R_0603, F.Cu at (115.9, 115.5)
- added R1509: 20.5k, 0_backbone:R_0603, F.Cu at (119.7, 115.5)
- added R1510: 4.02k, 0_backbone:R_0603, F.Cu at (123.6, 115.5)
- added R1511: 100k, 0_backbone:R_0603, F.Cu at (127.4, 115.5)
- added R1512: 27k, 0_backbone:R_0603, F.Cu at (104.3, 117.9)
- added R1513: 100k, 0_backbone:R_0603, F.Cu at (108.2, 117.9)
- added R201: 10k, 0_backbone:R_0603, F.Cu at (35.8, 36.0)
- added R301: 82k, 0_backbone:R_0603, F.Cu at (57.9, 33.9)
- added R302: 7.5k, 0_backbone:R_0603, F.Cu at (61.8, 33.9)
- added R303: 24.9k, 0_backbone:R_0603, F.Cu at (65.6, 33.9)
- added R304: 15k, 0_backbone:R_0603, F.Cu at (69.5, 33.9)
- added R305: 33.2k, 0_backbone:R_0603, F.Cu at (73.3, 33.9)
- added R306: 2.37k, 0_backbone:R_0603, F.Cu at (77.2, 33.9)
- added R307: 100, 0_backbone:R_0603, F.Cu at (81.0, 33.9)
- added R308: 2.2, 0_backbone:R_0603, F.Cu at (84.9, 33.9)
- added R309: 240, 0_backbone:R_0603, F.Cu at (88.7, 33.9)
- added R310: 20k, 0_backbone:R_0603, F.Cu at (92.6, 33.9)
- added R311: 4.7k, 0_backbone:R_0603, F.Cu at (49.8, 36.4)
- added R312: 2.2, 0_backbone:R_0603, F.Cu at (53.7, 36.4)
- added R401: 82k, 0_backbone:R_0603, F.Cu at (109.9, 30.5)
- added R402: 7.5k, 0_backbone:R_0603, F.Cu at (113.8, 30.5)
- added R403: 49.9k, 0_backbone:R_0603, F.Cu at (117.6, 30.5)
- added R404: 11k, 0_backbone:R_0603, F.Cu at (121.5, 30.5)
- added R405: 23.2k, 0_backbone:R_0603, F.Cu at (125.3, 30.5)
- added R406: 4.42k, 0_backbone:R_0603, F.Cu at (129.2, 30.5)
- added R407: 1k, 0_backbone:R_0603, F.Cu at (133.0, 30.5)
- added R408: 2.2, 0_backbone:R_0603, F.Cu at (136.9, 30.5)
- added R409: 150, 0_backbone:R_0603, F.Cu at (140.7, 30.5)
- added R410: 20k, 0_backbone:R_0603, F.Cu at (101.8, 33.0)
- added R411: 1k, 0_backbone:R_0603, F.Cu at (105.7, 33.0)
- added R412: 2.2, 0_backbone:R_0603, F.Cu at (109.5, 33.0)
- added R501: 442k, 0_backbone:R_0603, F.Cu at (173.5, 25.2)
- added R502: 90.9k, 0_backbone:R_0603, F.Cu at (177.4, 25.2)
- added R503: 243k, 0_backbone:R_0603, F.Cu at (181.2, 25.2)
- added R504: 16.9k, 0_backbone:R_0603, F.Cu at (185.1, 25.2)
- added R505: 53.6k, 0_backbone:R_0603, F.Cu at (149.8, 29.0)
- added R506: 10.2k, 0_backbone:R_0603, F.Cu at (153.7, 29.0)
- added R507: 1k, 0_backbone:R_0603, F.Cu at (157.5, 29.0)
- added R508: 453k, 0_backbone:R_0603, F.Cu at (161.4, 29.0)
- added R509: 100k, 0_backbone:R_0603, F.Cu at (165.2, 29.0)
- added R510: 1k, 0_backbone:R_0603, F.Cu at (169.1, 29.0)
- added R601: 910k, 0_backbone:R_0603, F.Cu at (141.9, 51.7)
- added R602: 200k, 0_backbone:R_0603, F.Cu at (145.7, 51.7)
- added R603: 1M, 0_backbone:R_0603, F.Cu at (149.6, 51.7)
- added R701: 10k, 0_backbone:R_0603, F.Cu at (106.0, 64.9)
- added R702: 9.53k, 0_backbone:R_0603, F.Cu at (109.8, 64.9)
- added R703: 90.9k, 0_backbone:R_0603, F.Cu at (113.7, 64.9)
- added R704: 10k, 0_backbone:R_0603, F.Cu at (117.5, 64.9)
- added R705: 10k, 0_backbone:R_0603, F.Cu at (121.4, 64.9)
- added R706: 10k, 0_backbone:R_0603, F.Cu at (125.2, 64.9)
- added R707: 10k, 0_backbone:R_0603, F.Cu at (129.1, 64.9)
- added R708: 1M, 0_backbone:R_0603, F.Cu at (93.8, 67.3)
- added R709: 82k, 0_backbone:R_0603, F.Cu at (97.7, 67.3)
- added R710: 100k, 0_backbone:R_0603, F.Cu at (101.5, 67.3)
- added R801: 16.9k, 0_backbone:R_0603, F.Cu at (149.9, 73.9)
- added R802: 10k, 0_backbone:R_0603, F.Cu at (153.8, 73.9)
- added R803: 1M, 0_backbone:R_0603, F.Cu at (157.6, 73.9)
- added R901: 16.9k, 0_backbone:R_0603, F.Cu at (149.9, 90.9)
- added R902: 10k, 0_backbone:R_0603, F.Cu at (153.8, 90.9)
- added R903: 1M, 0_backbone:R_0603, F.Cu at (157.6, 90.9)
- added TP1101: RESET, 0_backbone:TestPoint_Pad_D1.5mm, F.Cu at (82.3, 47.8)
- added TP1102: UART0_TXD, 0_backbone:TestPoint_Pad_D1.5mm, F.Cu at (86.0, 47.8)
- added TP1103: UART0_RXD, 0_backbone:TestPoint_Pad_D1.5mm, F.Cu at (49.8, 59.0)
- added TP1104: UART0_TNOW, 0_backbone:TestPoint_Pad_D1.5mm, F.Cu at (53.5, 59.0)
- added TP1105: UART1_TXD, 0_backbone:TestPoint_Pad_D1.5mm, F.Cu at (57.3, 59.0)
- added TP1106: UART1_RXD, 0_backbone:TestPoint_Pad_D1.5mm, F.Cu at (61.0, 59.0)
- added TP1107: UART1_TNOW, 0_backbone:TestPoint_Pad_D1.5mm, F.Cu at (64.8, 59.0)
- added TP1108: UART2_TXD, 0_backbone:TestPoint_Pad_D1.5mm, F.Cu at (68.5, 59.0)
- added TP1109: UART2_RXD, 0_backbone:TestPoint_Pad_D1.5mm, F.Cu at (72.3, 59.0)
- added TP1110: UART2_TNOW, 0_backbone:TestPoint_Pad_D1.5mm, F.Cu at (76.0, 59.0)
- added TP1111: UART3_TXD, 0_backbone:TestPoint_Pad_D1.5mm, F.Cu at (79.8, 59.0)
- added TP1112: UART3_RXD, 0_backbone:TestPoint_Pad_D1.5mm, F.Cu at (83.5, 59.0)
- added TP1113: UART3_TNOW, 0_backbone:TestPoint_Pad_D1.5mm, F.Cu at (49.8, 62.7)
- added TP1201: SHDN_485, 0_backbone:TestPoint_Pad_D1.5mm, F.Cu at (17.5, 105.9)
- added TP1202: TXD, 0_backbone:TestPoint_Pad_D1.5mm, F.Cu at (21.3, 105.9)
- added TP1203: RXD, 0_backbone:TestPoint_Pad_D1.5mm, F.Cu at (25.0, 105.9)
- added TP1204: TNOW, 0_backbone:TestPoint_Pad_D1.5mm, F.Cu at (28.8, 105.9)
- added TP1205: A, 0_backbone:TestPoint_Pad_D1.5mm, F.Cu at (3.77, 109.9)
- added TP1206: B, 0_backbone:TestPoint_Pad_D1.5mm, F.Cu at (7.53, 109.9)
- added TP1207: DATA, 0_backbone:TestPoint_Pad_D1.5mm, F.Cu at (11.3, 109.9)
- added TP1301: SHDN_485, 0_backbone:TestPoint_Pad_D1.5mm, F.Cu at (51.0, 105.9)
- added TP1302: TXD, 0_backbone:TestPoint_Pad_D1.5mm, F.Cu at (54.8, 105.9)
- added TP1303: RXD, 0_backbone:TestPoint_Pad_D1.5mm, F.Cu at (58.5, 105.9)
- added TP1304: TNOW, 0_backbone:TestPoint_Pad_D1.5mm, F.Cu at (62.3, 105.9)
- added TP1305: A, 0_backbone:TestPoint_Pad_D1.5mm, F.Cu at (37.3, 109.9)
- added TP1306: B, 0_backbone:TestPoint_Pad_D1.5mm, F.Cu at (41.0, 109.9)
- added TP1307: DATA, 0_backbone:TestPoint_Pad_D1.5mm, F.Cu at (44.8, 109.9)
- added TP1401: SHDN_485, 0_backbone:TestPoint_Pad_D1.5mm, F.Cu at (84.5, 105.9)
- added TP1402: TXD, 0_backbone:TestPoint_Pad_D1.5mm, F.Cu at (88.3, 105.9)
- added TP1403: RXD, 0_backbone:TestPoint_Pad_D1.5mm, F.Cu at (92.0, 105.9)
- added TP1404: TNOW, 0_backbone:TestPoint_Pad_D1.5mm, F.Cu at (95.8, 105.9)
- added TP1405: A, 0_backbone:TestPoint_Pad_D1.5mm, F.Cu at (70.8, 109.9)
- added TP1406: B, 0_backbone:TestPoint_Pad_D1.5mm, F.Cu at (74.5, 109.9)
- added TP1407: DATA, 0_backbone:TestPoint_Pad_D1.5mm, F.Cu at (78.3, 109.9)
- added TP1501: SHDN_485, 0_backbone:TestPoint_Pad_D1.5mm, F.Cu at (118.0, 105.9)
- added TP1502: TXD, 0_backbone:TestPoint_Pad_D1.5mm, F.Cu at (121.8, 105.9)
- added TP1503: RXD, 0_backbone:TestPoint_Pad_D1.5mm, F.Cu at (125.5, 105.9)
- added TP1504: TNOW, 0_backbone:TestPoint_Pad_D1.5mm, F.Cu at (129.3, 105.9)
- added TP1505: A, 0_backbone:TestPoint_Pad_D1.5mm, F.Cu at (104.3, 109.9)
- added TP1506: B, 0_backbone:TestPoint_Pad_D1.5mm, F.Cu at (108.0, 109.9)
- added TP1507: DATA, 0_backbone:TestPoint_Pad_D1.5mm, F.Cu at (111.8, 109.9)
- added TP201: +19V_IN, 0_backbone:TestPoint_Pad_D1.5mm, F.Cu at (24.1, 36.7)
- added TP202: +19V_JETSON, 0_backbone:TestPoint_Pad_D1.5mm, F.Cu at (27.9, 36.7)
- added TP301: PGOOD, 0_backbone:TestPoint_Pad_D1.5mm, F.Cu at (64.9, 30.5)
- added TP302: +12V_SERVO, 0_backbone:TestPoint_Pad_D1.5mm, F.Cu at (68.7, 30.5)
- added TP401: PGOOD, 0_backbone:TestPoint_Pad_D1.5mm, F.Cu at (111.1, 27.4)
- added TP402: +5V_SERVO, 0_backbone:TestPoint_Pad_D1.5mm, F.Cu at (114.8, 27.4)
- added TP501: +5V_USB, 0_backbone:TestPoint_Pad_D1.5mm, F.Cu at (149.8, 25.9)
- added TP502: +3V3, 0_backbone:TestPoint_Pad_D1.5mm, F.Cu at (153.5, 25.9)
- added TP601: DIR, 0_backbone:TestPoint_Pad_D1.5mm, F.Cu at (154.6, 47.8)
- added TP701: GRSTz, 0_backbone:TestPoint_Pad_D1.5mm, F.Cu at (107.7, 59.3)
- added TP702: VDD_HUB, 0_backbone:TestPoint_Pad_D1.5mm, F.Cu at (111.5, 59.3)
- added U1001: TPS2553DBVR, 0_backbone:SOT-23-6_L2.9-W1.6-P0.95-LS2.8-BR, F.Cu at (138.4, 104.2)
- added U1101: CH344Q, 0_backbone:LQFP-48_L7.0-W7.0-P0.50-LS9.0-BL, F.Cu at (53.5, 51.5)
- added U1201: SP3485EN-L/TR, 0_backbone:SOIC-8_L5.0-W4.0-P1.27-LS6.0-BL, F.Cu at (13.8, 94.0)
- added U1202: SN74LVC2G241DCU, 0_backbone:VSSOP-8_L2.3-W2.0-P0.50-LS3.1-BR, F.Cu at (4.35, 105.8)
- added U1203: TPS16630PWPR, 0_backbone:HTSSOP-20_L6.5-W4.4-P0.65-LS6.4-TL-EP2.58, F.Cu at (6.32, 93.9)
- added U1204: TPS25961DRVR, 0_backbone:WSON-6_L2.0-W2.0-P0.65-TL-EP, F.Cu at (13.7, 105.8)
- added U1301: SP3485EN-L/TR, 0_backbone:SOIC-8_L5.0-W4.0-P1.27-LS6.0-BL, F.Cu at (47.3, 94.0)
- added U1302: SN74LVC2G241DCU, 0_backbone:VSSOP-8_L2.3-W2.0-P0.50-LS3.1-BR, F.Cu at (37.9, 105.8)
- added U1303: TPS16630PWPR, 0_backbone:HTSSOP-20_L6.5-W4.4-P0.65-LS6.4-TL-EP2.58, F.Cu at (39.8, 93.9)
- added U1304: TPS25961DRVR, 0_backbone:WSON-6_L2.0-W2.0-P0.65-TL-EP, F.Cu at (47.2, 105.8)
- added U1401: SP3485EN-L/TR, 0_backbone:SOIC-8_L5.0-W4.0-P1.27-LS6.0-BL, F.Cu at (80.8, 94.0)
- added U1402: SN74LVC2G241DCU, 0_backbone:VSSOP-8_L2.3-W2.0-P0.50-LS3.1-BR, F.Cu at (71.4, 105.8)
- added U1403: TPS16630PWPR, 0_backbone:HTSSOP-20_L6.5-W4.4-P0.65-LS6.4-TL-EP2.58, F.Cu at (73.3, 93.9)
- added U1404: TPS25961DRVR, 0_backbone:WSON-6_L2.0-W2.0-P0.65-TL-EP, F.Cu at (80.7, 105.8)
- added U1501: SP3485EN-L/TR, 0_backbone:SOIC-8_L5.0-W4.0-P1.27-LS6.0-BL, F.Cu at (114.3, 94.0)
- added U1502: SN74LVC2G241DCU, 0_backbone:VSSOP-8_L2.3-W2.0-P0.50-LS3.1-BR, F.Cu at (104.9, 105.8)
- added U1503: TPS16630PWPR, 0_backbone:HTSSOP-20_L6.5-W4.4-P0.65-LS6.4-TL-EP2.58, F.Cu at (106.8, 93.9)
- added U1504: TPS25961DRVR, 0_backbone:WSON-6_L2.0-W2.0-P0.65-TL-EP, F.Cu at (114.2, 105.8)
- added U201: LM74700QDBVRQ1, 0_backbone:SOT-23-6_L2.9-W1.6-P0.95-LS2.8-BL, F.Cu at (38.3, 27.8)
- added U301: LM5145RGYR, 0_backbone:VQFN-20_L4.5-W3.5-P0.50-BL-EP, F.Cu at (58.5, 18.7)
- added U401: LM5145RGYR, 0_backbone:VQFN-20_L4.5-W3.5-P0.50-BL-EP, F.Cu at (103.7, 18.7)
- added U501: TPS54560DDAR, 0_backbone:SOIC-8_L5.0-W4.0-P1.27-LS6.0-BL-EP2.0, F.Cu at (174.8, 6.29)
- added U502: TLV62569DBVR, 0_backbone:SOT-23-5_L3.0-W1.7-P0.95-LS2.8-BR, F.Cu at (163.3, 21.7)
- added U601: HD3SS3220RNHR, 0_backbone:WQFN-30_L4.5-W2.5-P0.4-BL-EP, F.Cu at (139.0, 48.0)
- added U701: TUSB8041IRGCR, 0_backbone:QFN-64_L9.0-W9.0-P0.50-BL-EP7.2, F.Cu at (97.3, 51.3)
- added U702: TLV62569DBVR, 0_backbone:SOT-23-5_L3.0-W1.7-P0.95-LS2.8-BR, F.Cu at (116.8, 48.1)
- added U801: TPS2553DBVR, 0_backbone:SOT-23-6_L2.9-W1.6-P0.95-LS2.8-BR, F.Cu at (138.4, 70.2)
- added U901: TPS2553DBVR, 0_backbone:SOT-23-6_L2.9-W1.6-P0.95-LS2.8-BR, F.Cu at (138.4, 87.2)
- added Y1101: 8MHz 20pF, 0_backbone:CRYSTAL-SMD_L5.0-W3.2, F.Cu at (62.7, 48.3)
- added Y701: 24MHz 18pF, 0_backbone:OSC-SMD_4P-L3.2-W2.5-BL, F.Cu at (111.8, 48.1)
Other:
- board outline added: 190 x 130 mm
- board text added: "${KKH_VERSION_DATE}"
- board text added: "JLCJLCJLCJLC"
- board text added: "ROBOT BACKBONE rev A"
- board text added: "buck-12v-servo"
- board text added: "buck-5v-servo"
- board text added: "buck-5v-usb"
- board text added: "input"
- board text added: "servo-port-0"
- board text added: "servo-port-1"
- board text added: "servo-port-2"
- board text added: "servo-port-3"
- board text added: "servo-uart"
- board text added: "usb-hub"
- board text added: "usb-port-1"
- board text added: "usb-port-2"
- board text added: "usb-port-3"
- board text added: "usbc-upstream"

Commit message: schematics
Parts:
- moved H104 52.7 mm to (200.7, 75.1)
- moved H103 52.2 mm to (19.2, 75.4)
- moved C201 30.3 mm to (48.2, 61.5)
- moved C203 30.2 mm to (55.0, 22.5)
- moved R201 27.5 mm to (56.2, 54.5)
- moved C206 27.4 mm to (46.5, 56.5)
- moved Q201 25.0 mm to (54.4, 34.3)
- moved TP202 24.5 mm to (40.0, 58.0)
- moved D202 23.7 mm to (52.9, 51.0)
- moved U201 23.5 mm to (56.2, 43.0)
- moved C1501 20.7 mm to (130.3, 123.9)
- moved C1503 20.7 mm to (138.4, 123.9)
- moved C1508 20.7 mm to (133.5, 98.6)
- moved C415 20.7 mm to (129.2, 37.9)
- moved C702 20.7 mm to (134.2, 73.3)
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Other:
- board size 190 x 130 mm -> 190 x 65 mm
