File: backbone/backbone.kicad_sch (KiCad schematic)
At the start: 0 parts

Commit message: update
Other:
- added sheet buck-12v-servo (buck-12v-servo.kicad_sch)
- added sheet buck-5v-servo (buck-5v-servo.kicad_sch)
- added sheet buck-5v-usb (buck-5v-usb.kicad_sch)
- added sheet input (input.kicad_sch)
- added sheet servo-port-0 (servo-port.kicad_sch)
- added sheet servo-port-1 (servo-port.kicad_sch)
- added sheet servo-port-2 (servo-port.kicad_sch)
- added sheet servo-port-3 (servo-port.kicad_sch)
- added sheet servo-uart (servo-uart.kicad_sch)
- added sheet usb-hub (usb-hub.kicad_sch)
- added sheet usb-port-1 (usb-port.kicad_sch)
- added sheet usb-port-2 (usb-port.kicad_sch)
- added sheet usb-port-3 (usb-port.kicad_sch)
- added sheet usbc-upstream (usbc-upstream.kicad_sch)
- note added: "ROBOT BACKBONE — root sheet = block diagram (FUNCTIONAL.md §3). Only sheet symbols live here; draw inside the sub-sheets. Sheets: 2 input · 3 buck-12v-servo · 4 buck-5v-servo · 5 buck-5v-usb · 6 usbc-upstream · 7 usb-hub · 8-10 usb-port-1..3 (one file) · 11 servo-uart · 12-15 servo-port-0..3 (one file) Rails are global power symbols: +19V_IN +19V_JETSON +12V_SERVO +5V_SERVO +5V_USB +3V3 +1V1_HUB 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"
- title: (none) -> Robot backbone — root (block diagram)

Commit message: before hand editing
Parts:
- added H101, H102, H103, H104: M3, 0_backbone:MountingHole_3.2mm_M3_Pad_Via, symbol 0_backbone:MountingHole
Other:
- note added: "Mounting holes (M3, pad + vias)"
- note added: "ROBOT BACKBONE — root sheet = block diagram (FUNCTIONAL.md §3). Sheet symbols plus the mechanical items (mounting holes) live here; everything electrical is in the sub-sheets. Sheets: 2 input · 3 buck-12v-servo · 4 buck-5v-servo · 5 buck-5v-usb · 6 usbc-upstream · 7 usb-hub · 8-10 usb-port-1..3 (one file) · 11 servo-uart · 12-15 servo-port-0..3 (one file) Rails are global power symbols from the p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"
- note removed: "ROBOT BACKBONE — root sheet = block diagram (FUNCTIONAL.md §3). Only sheet symbols live here; draw inside the sub-sheets. Sheets: 2 input · 3 buck-12v-servo · 4 buck-5v-servo · 5 buck-5v-usb · 6 usbc-upstream · 7 usb-hub · 8-10 usb-port-1..3 (one file) · 11 servo-uart · 12-15 servo-port-0..3 (one file) Rails are global power symbols: +19V_IN +19V_JETSON +12V_SERVO +5V_SERVO +5V_USB +3V3 +1V1_HUB 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"
