File: backbone/buck-12v-servo.kicad_sch (KiCad schematic)
At the start: 0 parts

Commit message: before hand editing
Parts:
- added C301: 33nF, 0_backbone:C_0603, symbol 0_backbone:C_0603
- added C302: 3.3nF, 0_backbone:C_0603, symbol 0_backbone:C_0603
- added C303: 47pF, 0_backbone:C_0603, symbol 0_backbone:C_0603
- added C304: 680pF, 0_backbone:C_0603, symbol 0_backbone:C_0603
- added C305: 2.2uF, 0_backbone:C_0603, symbol 0_backbone:C_0603
- added C306: 100nF, 0_backbone:C_0603, symbol 0_backbone:C_0603
- added C307: 100nF 100V, 0_backbone:C_0805, symbol 0_backbone:C_0805
- added C308: 10pF, 0_backbone:C_0603, symbol 0_backbone:C_0603
- added C309, C310, C311, C312, C313: 4.7uF 100V, 0_backbone:C1210, symbol 0_backbone:C3225X7S2A475KT000N
- added C314, C315, C316, C317: 47uF 16V, 0_backbone:C1210, symbol 0_backbone:GRM32ER61C476KE15L
- added C318, C319: 22uF 25V, 0_backbone:C1210, symbol 0_backbone:CS3225X7R226K250NRL
- added C320, C321: 470uF 25V, 0_backbone:CAP-SMD_BD8.0-L8.3-W8.3-LS9.0-FD_H10.5, symbol 0_backbone:MA25V470M8X10
- added C322: 100pF, 0_backbone:C_0603, symbol 0_backbone:C_0603
- added D301: SS14, 0_backbone:D_SMA, symbol 0_backbone:SS14
- added D302: LED Green, 0_backbone:D_0805, symbol 0_backbone:LED_0805_Green
- added JP301: SYNCIN: 1-2 GND=DEM, 2-3 VCC=FPWM, 0_backbone:SolderJumper-3_P1.3mm_Bridged12_RoundedPad1.0x1.5mm, symbol 0_backbone:SolderJumper_3_Bridged12
- added L301: 4.7uH 20A, 0_backbone:IND-SMD_L13.5-W12.6, symbol 0_backbone:TMPA1265SP-4R7MN-D
- added Q301, Q302: CSD18532Q5B, 0_backbone:SON-8_L5.0-W6.0-P1.27-BL-1, symbol 0_backbone:CSD18532Q5B
- added R301: 82k, 0_backbone:R_0603, symbol 0_backbone:R_0603
- added R302: 7.5k, 0_backbone:R_0603, symbol 0_backbone:R_0603
- added R303: 24.9k, 0_backbone:R_0603, symbol 0_backbone:R_0603
- added R304: 15k, 0_backbone:R_0603, symbol 0_backbone:R_0603
- added R305: 33.2k, 0_backbone:R_0603, symbol 0_backbone:R_0603
- added R306: 2.37k, 0_backbone:R_0603, symbol 0_backbone:R_0603
- added R307: 100, 0_backbone:R_0603, symbol 0_backbone:R_0603
- added R308, R312: 2.2, 0_backbone:R_0603, symbol 0_backbone:R_0603
- added R309: 240, 0_backbone:R_0603, symbol 0_backbone:R_0603
- added R310: 20k, 0_backbone:R_0603, symbol 0_backbone:R_0603
- added R311: 4.7k, 0_backbone:R_0603, symbol 0_backbone:R_0603
- added TP301: PGOOD, 0_backbone:TestPoint_Pad_D1.5mm, symbol 0_backbone:TestPoint
- added TP302: +12V_SERVO, 0_backbone:TestPoint_Pad_D1.5mm, symbol 0_backbone:TestPoint
- added U301: LM5145RGYR, 0_backbone:VQFN-20_L4.5-W3.5-P0.50-BL-EP, symbol 0_backbone:LM5145RGYR
Connections:
- net +12V_SERVO: now also C314.1, C315.1, C316.1, C317.1, C318.1, C319.1, C320.1, C321.1, D301.2, L301.2, R305.1, R307.1, R311.1, TP302.1
- new net: D302.2, R311.2
- new net: C322.1, R312.2
- new net: C304.1, R307.2
- new net: C306.1, R308.2
- new net: C302.1, R304.2
- new net +19V_IN: C307.1, C309.1, C310.1, C311.1, C312.1, C313.1, Q301.5 (D), Q301.6 (D), Q301.7 (D), Q301.8 (D), Q301.9 (EP), R301.1, U301.20 (VIN)
- new net BOOT: R308.1, U301.17 (BST)
- new net COMP: C303.1, R304.1, U301.4 (COMP)
- new net FB: C302.2, C303.2, C304.2, R305.2, R306.1, U301.5 (FB)
- new net GND: C301.2, C305.2, C307.2, C308.2, C309.2, C310.2, C311.2, C312.2, C313.2, C314.2, C315.2, C316.2, C317.2, C318.2, C319.2, C320.2, C321.2, C322.2, D302.1, JP301.1 (A), Q302.1 (S), Q302.2 (S), Q302.3 (S), R302.2, R303.2, R306.2, U301.12 (PGND), U301.15 (EP), U301.21 (EP), U301.6 (AGND)
- new net HO: Q301.4 (G), U301.18 (HO)
- new net ILIM: C308.1, R309.1, U301.11 (ILIM)
- new net LO: Q302.4 (G), U301.13 (LO)
- new net PGOOD: R310.2, TP301.1, U301.10 (PGOOD)
- new net RT: R303.1, U301.2 (RT)
- new net SS: C301.1, U301.3 (SS/TRK)
- new net SW: C306.2, L301.1, Q301.1 (S), Q301.2 (S), Q301.3 (S), Q302.5 (D), Q302.6 (D), Q302.7 (D), Q302.8 (D), Q302.9 (EP), R309.2, R312.1, U301.19 (SW)
- new net SYNCIN: JP301.2 (C), U301.8 (SYNCIN)
- new net UVLO: R301.2, R302.1, U301.1 (EN/UVLO)
- new net VCC: C305.1, D301.1, JP301.3 (B), R310.1, U301.14 (VCC)
- no-connect marks 0 -> 1
Other:
- note added: "BUCK A — +12V_SERVO, 15 A continuous, 400 kHz. Copy of TI LM5145 datasheet Application Circuit 2 (12 V/10 A, 14.4-48 V in) with the power stage uprated: Q1/Q2 CSD18532Q5B (60 V, 2.5 mΩ), 4.7 µH 25 A inductor, 5 × 4.7 µF/100 V in, 4 × 47 µF + 2 × 22 µF + 2 × 470 µF polymer out. RILIM 240 Ω with 2.5 mΩ RDS(on) sets the valley current limit near 19 A (ILIM sources 200 µA in RDS(on) mode); CILIM to P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"
- note added: "CIN: 100 V ceramics (plus the bulk bank on the input sheet)"
- note added: "COUT: ceramics + polymer bulk bank (shared by all four ports)"
- note added: "LM5145 controller"
- note added: "Optional SW-node RC snubber (DNP until the SW ringing is measured)"
- note added: "Power stage: Q1 high side, Q2 low side, inductor, output bank"
- note added: "UVLO, frequency, soft-start, compensation (type III)"
- note added: "VCC, bootstrap, current limit, PGOOD, SYNCIN mode"
- note removed: "BUCK A — +12V_SERVO, 10–20 A, LM5145 controller + external FETs Golden reference: datasheets/reference/ti-snvu545-lm5145evm-hd-20a.pdf (copy the EVM layout), datasheets/lm5145.pdf WEBENCH design still to collect (datasheets/README.md) — currents follow decision D1. Parts (LCSC): LM5145RGYR C485912; FETs, inductor, caps from the WEBENCH BOM Consumes: +19V_IN, GND. Produces: +12V_SERVO (shared bulk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"

Commit message: schematics
Connections:
- net GND: now also C301.1, R302.1, R303.1; no longer C301.2, R302.2, R303.2
- net SW: no longer C306.2, L301.1, Q301.1 (S), Q301.2 (S), Q301.3 (S), Q302.5 (D), Q302.6 (D), Q302.7 (D), Q302.8 (D), Q302.9 (EP), R309.2, U301.19 (SW)
- net at R308.2: now also U301.17 (BST); no longer C306.1
- net at C302.1: now also C303.1, C304.2, R305.2, R306.1, U301.5 (FB); no longer R304.2
- net BOOT: no longer names the net of R308.1
- net BOOT: now also C306.1; no longer U301.17 (BST)
- removed net COMP: C303.1, R304.1, U301.4 (COMP)
- removed net FB: C302.2, C303.2, C304.2, R305.2, R306.1, U301.5 (FB)
- net HO: no longer names the net of Q301.4 (G), U301.18 (HO)
- net ILIM: no longer names the net of C308.1, R309.1, U301.11 (ILIM)
- net LO: no longer names the net of Q302.4 (G), U301.13 (LO)
- net PGOOD: no longer names the net of R310.2, TP301.1, U301.10 (PGOOD)
- net RT: no longer names the net of U301.2 (RT)
- net RT: now also R303.2; no longer R303.1
- net SS: no longer names the net of U301.3 (SS/TRK)
- net SS: now also C301.2; no longer C301.1
- net SYNCIN: no longer names the net of JP301.2 (C), U301.8 (SYNCIN)
- net UVLO: no longer names the net of R301.2, U301.1 (EN/UVLO)
- net UVLO: now also R302.2; no longer R302.1
- net VCC: no longer names the net of C305.1, D301.1, JP301.3 (B), R310.1, U301.14 (VCC)
- new net: C303.2, R304.2, U301.4 (COMP)
- new net: C306.2, L301.1, Q301.1 (S), Q301.2 (S), Q301.3 (S), Q302.5 (D), Q302.6 (D), Q302.7 (D), Q302.8 (D), Q302.9 (EP), R309.2, U301.19 (SW)
- new net: C302.2, R304.1
Other:
- note added: "Optional SW-node RC snubber"
- note removed: "Optional SW-node RC snubber (DNP until the SW ringing is measured)"
- note removed: "Power stage: Q1 high side, Q2 low side, inductor, output bank"
- note removed: "UVLO, frequency, soft-start, compensation (type III)"
- note removed: "VCC, bootstrap, current limit, PGOOD, SYNCIN mode"
- moved on the sheet: C301, C302, C303, C304, C305, C306, C307, C308, C309, C310, C311, C312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
