File: backbone/buck-5v-servo.kicad_sch (KiCad schematic)
At the start: 0 parts

Commit message: before hand editing
Parts:
- added C401: 47nF, 0_backbone:C_0603, symbol 0_backbone:C_0603
- added C402: 4.7nF, 0_backbone:C_0603, symbol 0_backbone:C_0603
- added C403: 150pF, 0_backbone:C_0603, symbol 0_backbone:C_0603
- added C404: 1.8nF, 0_backbone:C_0603, symbol 0_backbone:C_0603
- added C405: 2.2uF, 0_backbone:C_0603, symbol 0_backbone:C_0603
- added C406: 100nF, 0_backbone:C_0603, symbol 0_backbone:C_0603
- added C407: 100nF 100V, 0_backbone:C_0805, symbol 0_backbone:C_0805
- added C408: 15pF, 0_backbone:C_0603, symbol 0_backbone:C_0603
- added C409, C410, C411, C412, C413: 2.2uF 100V, 0_backbone:C1210, symbol 0_backbone:C3225X7R2A225KT5L0U
- added C414, C415, C416, C417, C418, C419: 47uF 10V, 0_backbone:C_1206, symbol 0_backbone:C_1206
- added C420: 470uF 10V, 0_backbone:CAP-SMD_BD6.3-L6.6-W6.6-LS7.3-FD-H7.7, symbol 0_backbone:MA10V470M6X8
- added C421: 100pF, 0_backbone:C_0603, symbol 0_backbone:C_0603
- added D401: LED Green, 0_backbone:D_0805, symbol 0_backbone:LED_0805_Green
- added JP401: SYNCIN: 1-2 GND=DEM, 2-3 VCC=FPWM, 0_backbone:SolderJumper-3_P1.3mm_Bridged12_RoundedPad1.0x1.5mm, symbol 0_backbone:SolderJumper_3_Bridged12
- added L401: 3.3uH 18A, 0_backbone:IND-SMD_L13.5-W12.6_125CDMCC-DS, symbol 0_backbone:TMPC1265HP-3R3MG-D
- added Q401, Q402: CSD18532Q5B, 0_backbone:SON-8_L5.0-W6.0-P1.27-BL-1, symbol 0_backbone:CSD18532Q5B
- added R401: 82k, 0_backbone:R_0603, symbol 0_backbone:R_0603
- added R402: 7.5k, 0_backbone:R_0603, symbol 0_backbone:R_0603
- added R403: 49.9k, 0_backbone:R_0603, symbol 0_backbone:R_0603
- added R404: 11k, 0_backbone:R_0603, symbol 0_backbone:R_0603
- added R405: 23.2k, 0_backbone:R_0603, symbol 0_backbone:R_0603
- added R406: 4.42k, 0_backbone:R_0603, symbol 0_backbone:R_0603
- added R407, R411: 1k, 0_backbone:R_0603, symbol 0_backbone:R_0603
- added R408, R412: 2.2, 0_backbone:R_0603, symbol 0_backbone:R_0603
- added R409: 150, 0_backbone:R_0603, symbol 0_backbone:R_0603
- added R410: 20k, 0_backbone:R_0603, symbol 0_backbone:R_0603
- added TP401: PGOOD, 0_backbone:TestPoint_Pad_D1.5mm, symbol 0_backbone:TestPoint
- added TP402: +5V_SERVO, 0_backbone:TestPoint_Pad_D1.5mm, symbol 0_backbone:TestPoint
- added U401: LM5145RGYR, 0_backbone:VQFN-20_L4.5-W3.5-P0.50-BL-EP, symbol 0_backbone:LM5145RGYR
Connections:
- net +5V_SERVO: now also C414.1, C415.1, C416.1, C417.1, C418.1, C419.1, C420.1, L401.2, R405.1, R407.1, R411.1, TP402.1
- new net: C421.1, R412.2
- new net: C406.1, R408.2
- new net: C404.1, R407.2
- new net: D401.2, R411.2
- new net: C402.1, R404.2
- new net +19V_IN: C407.1, C409.1, C410.1, C411.1, C412.1, C413.1, Q401.5 (D), Q401.6 (D), Q401.7 (D), Q401.8 (D), Q401.9 (EP), R401.1, U401.20 (VIN)
- new net BOOT: R408.1, U401.17 (BST)
- new net COMP: C403.1, R404.1, U401.4 (COMP)
- new net FB: C402.2, C403.2, C404.2, R405.2, R406.1, U401.5 (FB)
- new net GND: C401.2, C405.2, C407.2, C408.2, C409.2, C410.2, C411.2, C412.2, C413.2, C414.2, C415.2, C416.2, C417.2, C418.2, C419.2, C420.2, C421.2, D401.1, JP401.1 (A), Q402.1 (S), Q402.2 (S), Q402.3 (S), R402.2, R403.2, R406.2, U401.12 (PGND), U401.15 (EP), U401.21 (EP), U401.6 (AGND)
- new net HO: Q401.4 (G), U401.18 (HO)
- new net ILIM: C408.1, R409.1, U401.11 (ILIM)
- new net LO: Q402.4 (G), U401.13 (LO)
- new net PGOOD: R410.2, TP401.1, U401.10 (PGOOD)
- new net RT: R403.1, U401.2 (RT)
- new net SS: C401.1, U401.3 (SS/TRK)
- new net SW: C406.2, L401.1, Q401.1 (S), Q401.2 (S), Q401.3 (S), Q402.5 (D), Q402.6 (D), Q402.7 (D), Q402.8 (D), Q402.9 (EP), R409.2, R412.1, U401.19 (SW)
- new net SYNCIN: JP401.2 (C), U401.8 (SYNCIN)
- new net UVLO: R401.2, R402.1, U401.1 (EN/UVLO)
- new net VCC: C405.1, JP401.3 (B), R410.1, U401.14 (VCC)
- no-connect marks 0 -> 1
Other:
- note added: "BUCK B — +5V_SERVO, 10 A continuous, 200 kHz. Copy of TI LM5145 datasheet Application Circuit 1 (5 V/20 A) and the LM5145EVM-HD-20A: same controller passives, Q1/Q2 CSD18532Q5B, 3.3 µH 30 A inductor, 5 × 2.2 µF/100 V in, 6 × 47 µF/10 V + 470 µF/10 V polymer out. RILIM 150 Ω with 2.5 mΩ RDS(on) → valley current limit near 12 A. Separate sheet on purpose: values differ and D1 option (b) deletes thi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"
- note added: "CIN: 100 V ceramics (plus the bulk bank on the input sheet)"
- note added: "COUT: ceramics + polymer bulk bank (shared by all four ports)"
- note added: "LM5145 controller"
- note added: "Optional SW-node RC snubber (DNP until the SW ringing is measured)"
- note added: "Power stage: Q1 high side, Q2 low side, inductor, output bank"
- note added: "UVLO, frequency, soft-start, compensation (type III)"
- note added: "VCC, bootstrap, current limit, PGOOD, SYNCIN mode"
- note removed: "BUCK B — +5V_SERVO, 5–10 A, same LM5145 design as Buck A with the 5 V divider Separate sheet file on purpose: KiCad shares symbol values between sheet instances, and D1 option (b) deletes this rail entirely. Golden reference: datasheets/reference/ti-snvu545-lm5145evm-hd-20a.pdf, datasheets/lm5145.pdf Consumes: +19V_IN, GND. Produces: +5V_SERVO — NEVER merged with +5V_USB (HARDWARE.md §5). Name th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"

Commit message: schematics
Connections:
- net VCC is gone; now on net +5V_SERVO: C405.1, JP401.3 (B), R410.1, U401.14 (VCC)
- net SW: no longer C406.2, L401.1, Q401.1 (S), Q401.2 (S), Q401.3 (S), Q402.5 (D), Q402.6 (D), Q402.7 (D), Q402.8 (D), Q402.9 (EP), R409.2, U401.19 (SW)
- net BOOT: no longer names the net of R408.1, U401.17 (BST)
- net COMP: no longer names the net of C403.1, R404.1, U401.4 (COMP)
- net FB: no longer names the net of C402.2, C403.2, C404.2, R405.2, R406.1, U401.5 (FB)
- net HO: no longer names the net of Q401.4 (G), U401.18 (HO)
- net ILIM: no longer names the net of C408.1, R409.1, U401.11 (ILIM)
- net LO: no longer names the net of Q402.4 (G), U401.13 (LO)
- net PGOOD: no longer names the net of R410.2, TP401.1, U401.10 (PGOOD)
- net RT: no longer names the net of R403.1, U401.2 (RT)
- net SS: no longer names the net of C401.1, U401.3 (SS/TRK)
- net SYNCIN: no longer names the net of JP401.2 (C), U401.8 (SYNCIN)
- net UVLO: no longer names the net of R401.2, R402.1, U401.1 (EN/UVLO)
- new net: C406.2, L401.1, Q401.1 (S), Q401.2 (S), Q401.3 (S), Q402.5 (D), Q402.6 (D), Q402.7 (D), Q402.8 (D), Q402.9 (EP), R409.2, U401.19 (SW)
Other:
- note added: "Optional SW-node RC snubber"
- note removed: "Optional SW-node RC snubber (DNP until the SW ringing is measured)"
- note removed: "Power stage: Q1 high side, Q2 low side, inductor, output bank"
- note removed: "UVLO, frequency, soft-start, compensation (type III)"
- note removed: "VCC, bootstrap, current limit, PGOOD, SYNCIN mode"
- moved on the sheet: C401, C402, C403, C404, C405, C406, C407, C408, C409, C410, C411, C412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
