File: backbone/buck-5v-usb.kicad_sch (KiCad schematic)
At the start: 0 parts

Commit message: before hand editing
Parts:
- added C501: 4.7nF, 0_backbone:C_0603, symbol 0_backbone:C_0603
- added C502: 47pF, 0_backbone:C_0603, symbol 0_backbone:C_0603
- added C503: 100nF, 0_backbone:C_0603, symbol 0_backbone:C_0603
- added C504, C505, C506, C507: 2.2uF 100V, 0_backbone:C1210, symbol 0_backbone:C3225X7R2A225KT5L0U
- added C508, C509, C510: 47uF 16V, 0_backbone:C1210, symbol 0_backbone:GRM32ER61C476KE15L
- added C511: 6.8pF, 0_backbone:C_0603, symbol 0_backbone:C_0603
- added C512: 4.7uF, 0_backbone:C_0805, symbol 0_backbone:C_0805
- added C513: 22uF, 0_backbone:C_0805, symbol 0_backbone:C_0805
- added D501: B560C, 0_backbone:SMC_L7.1-W6.2-LS8.1-RD, symbol 0_backbone:B560C-13-F
- added D502, D503: LED Green, 0_backbone:D_0805, symbol 0_backbone:LED_0805_Green
- added L501: 7.2uH 6A, 0_backbone:IND-SMD_L10.2-W10.2_7447798720, symbol 0_backbone:7447798720
- added L502: 2.2uH 3.4A, 0_backbone:IND-SMD_L4.0-W4.0_LQH44PN2R2MP0L, symbol 0_backbone:SMNR4020-2.2UH
- added R501: 442k, 0_backbone:R_0603, symbol 0_backbone:R_0603
- added R502: 90.9k, 0_backbone:R_0603, symbol 0_backbone:R_0603
- added R503: 243k, 0_backbone:R_0603, symbol 0_backbone:R_0603
- added R504: 16.9k, 0_backbone:R_0603, symbol 0_backbone:R_0603
- added R505: 53.6k, 0_backbone:R_0603, symbol 0_backbone:R_0603
- added R506: 10.2k, 0_backbone:R_0603, symbol 0_backbone:R_0603
- added R507, R510: 1k, 0_backbone:R_0603, symbol 0_backbone:R_0603
- added R508: 453k, 0_backbone:R_0603, symbol 0_backbone:R_0603
- added R509: 100k, 0_backbone:R_0603, symbol 0_backbone:R_0603
- added TP501: +5V_USB, 0_backbone:TestPoint_Pad_D1.5mm, symbol 0_backbone:TestPoint
- added TP502: +3V3, 0_backbone:TestPoint_Pad_D1.5mm, symbol 0_backbone:TestPoint
- added U501: TPS54560DDAR, 0_backbone:SOIC-8_L5.0-W4.0-P1.27-LS6.0-BL-EP2.0, symbol 0_backbone:TPS54560DDAR
- added U502: TLV62569DBVR, 0_backbone:SOT-23-5_L3.0-W1.7-P0.95-LS2.8-BR, symbol 0_backbone:TLV62569DBVR
Connections:
- net +3V3: now also C511.1, C513.1, L502.2, R508.1, R510.1, TP502.1
- net +5V_USB: now also C508.1, C509.1, C510.1, C512.1, L501.2, R505.1, R507.1, TP501.1, U502.1 (EN), U502.4 (VIN)
- new net: C501.1, R504.2
- new net: D503.2, R510.2
- new net: D502.2, R507.2
- new net +19V_IN: C504.1, C505.1, C506.1, C507.1, R501.1, U501.2 (VIN)
- new net BOOT: C503.1, U501.1 (BOOT)
- new net COMP: C502.1, R504.1, U501.6 (COMP)
- new net EN: R501.2, R502.1, U501.3 (EN)
- new net FB: R505.2, R506.1, U501.5 (FB)
- new net FB_3V3: C511.2, R508.2, R509.1, U502.5 (FB)
- new net GND: C501.2, C502.2, C504.2, C505.2, C506.2, C507.2, C508.2, C509.2, C510.2, C512.2, C513.2, D501.2 (A), D502.1, D503.1, R502.2, R503.2, R506.2, R509.2, U501.7 (GND), U501.9 (EP), U502.2 (GND)
- new net RT: R503.1, U501.4 (RT/CLK)
- new net SW: C503.2, D501.1 (K), L501.1, U501.8 (SW)
- new net SW_3V3: L502.1, U502.3 (SW)
Other:
- note added: "BUCK C — +5V_USB (TPS54560, 5 A, 400 kHz) exactly as the TPS54560 datasheet 5 V design example / TPS54560EVM-515: EN divider 442 k / 90.9 k (UVLO ≈ 7 V on), RT 243 k, comp 16.9 k + 4.7 nF, 47 pF, FB 53.6 k / 10.2 k, 7.2 µH 6 A, B560C catch diode, 3 × 47 µF/16 V out. +3V3 — TLV62569 from the quiet +5V_USB rail (never the servo rails): 2.2 µH, 4.7 µF in, 22 µF out, FB 453 k / 100 k + 6.8 pF → 3.32 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"
- note added: "TLV62569: +5V_USB → +3V3"
- note added: "TPS54560: +19V_IN → +5V_USB"
- note removed: "BUCK C — +5V_USB (TPS54560, 5 A) and the quiet +3V3 rail (TLV62569 from +5V_USB) Golden reference: datasheets/reference/ti-slvu863-tps54560-evm.pdf, datasheets/tps54560.pdf, datasheets/tlv62569.pdf Parts (LCSC): TPS54560DDAR C31966, TLV62569DBVR C141836 Consumes: +19V_IN, GND. Produces: +5V_USB (3 × 1.5 A ports + 3V3), +3V3 (hub I/O, HD3SS3220, CH344Q, front-ends, < 0.5 A) Name the switch node SW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"

Commit message: schematics
Connections:
- net +5V_USB: no longer C512.1, L501.2, R505.1, R507.1, TP501.1, U502.1 (EN), U502.4 (VIN)
- net +3V3: no longer names the net of C511.1, C513.1, L502.2, R508.1, R510.1, TP502.1
- net BOOT: no longer names the net of C503.1, U501.1 (BOOT)
- net COMP: no longer names the net of C502.1, R504.1, U501.6 (COMP)
- net EN: no longer names the net of R501.2, R502.1, U501.3 (EN)
- net FB: no longer names the net of R505.2, R506.1, U501.5 (FB)
- net FB_3V3: no longer names the net of C511.2, R508.2, R509.1, U502.5 (FB)
- net RT: no longer names the net of R503.1, U501.4 (RT/CLK)
- net SW: no longer names the net of C503.2, D501.1 (K), L501.1, U501.8 (SW)
- net SW_3V3: no longer names the net of L502.1, U502.3 (SW)
- new net: C512.1, L501.2, R505.1, R507.1, TP501.1, U502.1 (EN), U502.4 (VIN)
Other:
- moved on the sheet: C501, C502, C503, C504, C505, C506, C507, C508, C509, C510, C511, C512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
