File: backbone/servo-port.kicad_sch (KiCad schematic)
At the start: 0 parts

Commit message: before hand editing
Parts:
- added C1201, C1202, C1203, C1204, C1206, C1207, C1209: 100nF, 0_backbone:C_0603, symbol 0_backbone:C_0603
- added C1205: 470uF 25V, 0_backbone:CAP-SMD_BD8.0-L8.3-W8.3-LS9.0-FD_H10.5, symbol 0_backbone:MA25V470M8X10
- added C1208: 470uF 10V, 0_backbone:CAP-SMD_BD6.3-L6.6-W6.6-LS7.3-FD-H7.7, symbol 0_backbone:MA10V470M6X8
- added D1201: PSM712-LF-T7, 0_backbone:SOT-23-3_L3.0-W1.7-P0.95-LS2.9-BR, symbol 0_backbone:PSM712
- added D1202: SMF5.0A, 0_backbone:D_SOD-123FL, symbol 0_backbone:SMF5.0A
- added D1203: SMBJ13A, 0_backbone:D_SMB, symbol 0_backbone:TVS_SMB
- added D1204: SMBJ6.0A, 0_backbone:D_SMB, symbol 0_backbone:TVS_SMB
- added J1201: RS-485 JST EH 4p, 0_backbone:CONN-TH_B4B-EH-A-LF-SN, symbol 0_backbone:B4B-EH-A
- added J1202: TTL JST EH 3p, 0_backbone:CONN-TH_B3B-EH-A-LF-SN, symbol 0_backbone:B3B-EH-A
- added JP1201: MODE: 1-2 RS-485 (default), 2-3 TTL, 0_backbone:SolderJumper-3_P1.3mm_Bridged12_RoundedPad1.0x1.5mm, symbol 0_backbone:SolderJumper_3_Bridged12
- added JP1202: MODE: bridged = auto-retry, open = latch-off, 0_backbone:SolderJumper-2_P1.3mm_Bridged_RoundedPad1.0x1.5mm, symbol 0_backbone:SolderJumper_2_Bridged
- added R1201, R1202, R1211, R1213: 100k, 0_backbone:R_0603, symbol 0_backbone:R_0603
- added R1203, R1206: 10k, 0_backbone:R_0603, symbol 0_backbone:R_0603
- added R1204: 120, 0_backbone:R_0603, symbol 0_backbone:R_0603
- added R1205: 22, 0_backbone:R_0603, symbol 0_backbone:R_0603
- added R1207: 249k, 0_backbone:R_0603, symbol 0_backbone:R_0603
- added R1208: 18.2k, 0_backbone:R_0603, symbol 0_backbone:R_0603
- added R1209: 20.5k, 0_backbone:R_0603, symbol 0_backbone:R_0603
- added R1210: 4.02k, 0_backbone:R_0603, symbol 0_backbone:R_0603
- added R1212: 27k, 0_backbone:R_0603, symbol 0_backbone:R_0603
- added TP1201: SHDN_485, 0_backbone:TestPoint_Pad_D1.5mm, symbol 0_backbone:TestPoint
- added TP1202: TXD, 0_backbone:TestPoint_Pad_D1.5mm, symbol 0_backbone:TestPoint
- added TP1203: RXD, 0_backbone:TestPoint_Pad_D1.5mm, symbol 0_backbone:TestPoint
- added TP1204: TNOW, 0_backbone:TestPoint_Pad_D1.5mm, symbol 0_backbone:TestPoint
- added TP1205: A, 0_backbone:TestPoint_Pad_D1.5mm, symbol 0_backbone:TestPoint
- added TP1206: B, 0_backbone:TestPoint_Pad_D1.5mm, symbol 0_backbone:TestPoint
- added TP1207: DATA, 0_backbone:TestPoint_Pad_D1.5mm, symbol 0_backbone:TestPoint
- added U1201: SP3485EN-L/TR, 0_backbone:SOIC-8_L5.0-W4.0-P1.27-LS6.0-BL, symbol 0_backbone:SP3485EN
- added U1202: SN74LVC2G241DCU, 0_backbone:VSSOP-8_L2.3-W2.0-P0.50-LS3.1-BR, symbol 0_backbone:SN74LVC2G241DCU
- added U1203: TPS16630PWPR, 0_backbone:HTSSOP-20_L6.5-W4.4-P0.65-LS6.4-TL-EP2.58, symbol 0_backbone:TPS16630PWPR
- added U1204: TPS25961DRVR, 0_backbone:WSON-6_L2.0-W2.0-P0.65-TL-EP, symbol 0_backbone:TPS25961DRVR
Connections:
- net RXD: now also R1203.2, TP1203.1, U1201.1 (RO), U1202.6 (1Y)
- net TNOW: now also JP1201.2 (C), TP1204.1, U1201.3 (DE), U1202.7 (2OE)
- net TXD: now also TP1202.1, U1201.4 (DI), U1202.5 (2A)
- new net +12V_SERVO: C1204.1, R1207.1, R1211.1, U1203.1 (IN), U1203.2 (IN), U1203.3 (IN), U1203.6 (P_IN)
- new net +3V3: C1201.1, C1202.1, R1201.1, R1202.1, R1203.1, R1206.1, U1201.8 (VCC), U1202.8 (VCC)
- new net +5V_SERVO: C1207.1, R1213.1, U1204.6 (IN)
- new net A: D1201.1 (A1), J1201.3, R1204.1, TP1205.1, U1201.6 (A)
- new net B: D1201.2 (A1), J1201.4, R1204.2, TP1206.1, U1201.7 (B)
- new net DATA: D1202.1, J1202.3, R1205.2, R1206.2, TP1207.1
- new net DATA_BUF: R1205.1, U1202.2 (1A), U1202.3 (2Y)
- new net DVDT_485: C1203.1, U1203.10 (dVdT)
- new net EN_TTL: R1213.2, U1204.5 (EN/UVLO)
- new net GND: C1201.2, C1202.2, C1203.2, C1204.2, C1205.2, C1206.2, C1207.2, C1208.2, C1209.2, D1201.3 (K), D1202.2, D1203.2, D1204.2, J1201.1, J1202.1, JP1202.2 (B), R1209.2, R1210.2, R1212.2, U1201.5 (GND), U1202.4 (GND), U1203.21 (EP), U1203.9 (GND), U1204.2 (OVLO), U1204.4 (GND), U1204.7 (GND)
- new net ILIM_485: R1210.1, U1203.11 (ILIM)
- new net ILIM_TTL: R1212.1, U1204.3 (ILIM)
- new net MODE_485: JP1202.1 (A), U1203.12 (MODE)
- new net OE_TTL: JP1201.3 (B), R1202.2, U1202.1 (~{1OE})
- new net OVP_485: R1207.2, R1208.1, U1203.8 (OVP)
- new net RE_485: JP1201.1 (A), R1201.2, U1201.2 (RE#)
- new net SHDN_485: R1211.2, TP1201.1, U1203.13 (~{SHDN})
- new net UVLO_485: R1208.2, R1209.1, U1203.7 (UVLO)
- new net VDD_485: C1205.1, C1206.1, D1203.1, J1201.2, U1203.18 (OUT), U1203.19 (OUT), U1203.20 (OUT)
- new net VDD_TTL: C1208.1, C1209.1, D1204.1, J1202.2, U1204.1 (OUT)
- no-connect marks 0 -> 3
Other:
- note added: "Front-end: RS-485 transceiver and TTL half-duplex buffer, mode select"
- note added: "Port power, RS-485 side: +12V_SERVO → TPS16630 e-fuse → VDD_485"
- note added: "Port power, TTL side: +5V_SERVO → TPS25961 e-fuse → VDD_TTL"
- note added: "RS-485 side (J1) and TTL side (J2)"
- note added: "SERVO PORT — one sheet, instantiated 4× as servo-port-0..3 (UART0..3). Everything replicated per port lives here. Front-end = ROBOTIS's RS-485 and 3.3 V TTL circuits with TNOW as TX_Enable: SP3485EN (DI = TXD, DE = TNOW, RE# = TNOW only when RS-485 is selected) and SN74LVC2G241 (2A = TXD → 2Y = DATA, 2OE = TNOW, 1A = DATA → 1Y = RXD, 1OE# = TNOW only when TTL is selected). Both receivers are off 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"
- note added: "Test points (bring-up)"
- note removed: "SERVO PORT — one sheet, instantiated 4× as servo-port-0..3. Contains everything replicated per port: front-end: SP3485EN C8963 (DI=TXD, DE=TNOW, R̄E̅=TNOW when RS-485 selected) + SN74LVC2G241 C10430 (2A=TXD, 2OE=TNOW, 1OE̅=TNOW when TTL selected, 1Y=RXD) mode select (D2): jumper / solder bridge routes TNOW to exactly ONE receiver enable; the other is tied inactive. Both receiver outputs wire-OR o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"
