File: backbone/servo-uart.kicad_sch (KiCad schematic)
At the start: 0 parts

Commit message: before hand editing
Parts:
- added C1101, C1102: 33pF, 0_backbone:C_0603, symbol 0_backbone:C_0603
- added C1103, C1104, C1105, C1106, C1107: 100nF, 0_backbone:C_0603, symbol 0_backbone:C_0603
- added C1108: 10uF, 0_backbone:C_0805, symbol 0_backbone:C_0805
- added D1101: LED ACT, 0_backbone:D_0805, symbol 0_backbone:LED_0805_Green
- added D1102: USBLC6-2SC6, 0_backbone:SOT-23-6_L2.9-W1.6-P0.95-LS2.8-BL, symbol 0_backbone:USBLC6-2SC6_C2687116
- added R1101: 10k, 0_backbone:R_0603, symbol 0_backbone:R_0603
- added R1102, R1103, R1104, R1105: 4.7k, 0_backbone:R_0603, symbol 0_backbone:R_0603
- added R1106: 1k, 0_backbone:R_0603, symbol 0_backbone:R_0603
- added TP1101: RESET, 0_backbone:TestPoint_Pad_D1.5mm, symbol 0_backbone:TestPoint
- added TP1102: UART0_TXD, 0_backbone:TestPoint_Pad_D1.5mm, symbol 0_backbone:TestPoint
- added TP1103: UART0_RXD, 0_backbone:TestPoint_Pad_D1.5mm, symbol 0_backbone:TestPoint
- added TP1104: UART0_TNOW, 0_backbone:TestPoint_Pad_D1.5mm, symbol 0_backbone:TestPoint
- added TP1105: UART1_TXD, 0_backbone:TestPoint_Pad_D1.5mm, symbol 0_backbone:TestPoint
- added TP1106: UART1_RXD, 0_backbone:TestPoint_Pad_D1.5mm, symbol 0_backbone:TestPoint
- added TP1107: UART1_TNOW, 0_backbone:TestPoint_Pad_D1.5mm, symbol 0_backbone:TestPoint
- added TP1108: UART2_TXD, 0_backbone:TestPoint_Pad_D1.5mm, symbol 0_backbone:TestPoint
- added TP1109: UART2_RXD, 0_backbone:TestPoint_Pad_D1.5mm, symbol 0_backbone:TestPoint
- added TP1110: UART2_TNOW, 0_backbone:TestPoint_Pad_D1.5mm, symbol 0_backbone:TestPoint
- added TP1111: UART3_TXD, 0_backbone:TestPoint_Pad_D1.5mm, symbol 0_backbone:TestPoint
- added TP1112: UART3_RXD, 0_backbone:TestPoint_Pad_D1.5mm, symbol 0_backbone:TestPoint
- added TP1113: UART3_TNOW, 0_backbone:TestPoint_Pad_D1.5mm, symbol 0_backbone:TestPoint
- added U1101: CH344Q, 0_backbone:LQFP-48_L7.0-W7.0-P0.50-LS9.0-BL, symbol 0_backbone:CH344Q_C2988084
- added Y1101: 8MHz 20pF, 0_backbone:CRYSTAL-SMD_L5.0-W3.2, symbol 0_backbone:Crystal_8MHz_5032
Connections:
- net DS4_DM: now also D1102.4 (I/O2)
- net DS4_DP: now also D1102.6 (I/O1)
- net UART0_RXD: now also TP1103.1, U1101.31 (RXD0)
- net UART0_TNOW: now also R1102.1, TP1104.1, U1101.39 (TNOW0/GPIO8)
- net UART0_TXD: now also TP1102.1, U1101.30 (TXD0)
- net UART1_RXD: now also TP1106.1, U1101.13 (RXD1)
- net UART1_TNOW: now also R1103.1, TP1107.1, U1101.18 (TNOW1/GPIO9)
- net UART1_TXD: now also TP1105.1, U1101.12 (TXD1)
- net UART2_RXD: now also TP1109.1, U1101.22 (RXD2)
- net UART2_TNOW: now also R1104.1, TP1110.1, U1101.19 (TNOW2/GPIO10)
- net UART2_TXD: now also TP1108.1, U1101.21 (TXD2)
- net UART3_RXD: now also TP1112.1, U1101.38 (RXD3)
- net UART3_TNOW: now also R1105.1, TP1113.1, U1101.34 (TNOW3/DTR3/GPIO11)
- net UART3_TXD: now also TP1111.1, U1101.37 (TXD3)
- new net: D1101.2, R1106.2
- new net +3V3: C1104.1, C1105.1, C1106.1, C1107.1, C1108.1, D1102.5 (VBUS), R1101.1, R1106.1, U1101.24 (VCC), U1101.36 (VCC), U1101.48 (VCC), U1101.9 (VCC)
- new net ACT: D1101.1, U1101.14 (ACT)
- new net GND: C1101.2, C1102.2, C1103.2, C1104.2, C1105.2, C1106.2, C1107.2, C1108.2, D1102.2 (GND), R1102.2, R1103.2, R1104.2, R1105.2, U1101.20 (GND), U1101.23 (GND), U1101.35 (GND), U1101.44 (TEST), U1101.47 (GND), U1101.8 (GND)
- new net RESET: C1103.1, R1101.2, TP1101.1, U1101.7 (RESET)
- new net UDM: D1102.3 (I/O2), U1101.42 (UD-)
- new net UDP: D1102.1 (I/O1), U1101.43 (UD+)
- new net XI: C1101.1, U1101.5 (XI), Y1101.1
- new net XO: C1102.1, U1101.6 (XO), Y1101.2
- no-connect marks 0 -> 19
Other:
- note added: "Crystal, reset, TNOW strap pull-downs, ACT LED"
- note added: "Decoupling (one 100 nF per VCC pin + 10 µF)"
- note added: "SERVO UART — CH344Q on hub port DS4 (USB 2.0 HS, UD+/UD- straight from the ESD array, no series resistors per WCH), four UARTs → servo-port-0..3. UART index ↔ physical port index is fixed by copper (software contract). 8 MHz ±0.4‰ crystal with 33 pF (20 pF CL), 100 nF on every VCC pin, TEST = GND. TNOW: a 4.7 k pull-down on each DTRx/TNOWx pin at power-up selects the TNOW function (CH344Q) and ke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"
- note added: "Test points (bring-up)"
- note added: "USB 2.0 ESD (hub DS4 ↔ CH344 UD+/UD-)"
- note removed: "SERVO UART — CH344Q, USB 2.0 from hub DS4, four UARTs → servo-port-0..3 (UART index ↔ port index is fixed: software contract) Golden reference: datasheets/ch344.pdf (CH344DS1, Chinese; TNOW facts in FUNCTIONAL.md §5.2) Parts (LCSC): CH344Q C2988084, USBLC6-2 C2687116 on DS4_DP/DM TNOW: DTRx/TNOWx/GPIOx pins (Q package 39, 18, 19, 34) become TNOW with a 4.7 kΩ pull-down at power-on. Add 10 kΩ pull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"

Commit message: schematics
Connections:
- net ACT: no longer names the net of D1101.1, U1101.14 (ACT)
- net RESET: no longer names the net of C1103.1, R1101.2, TP1101.1, U1101.7 (RESET)
- net UDM: no longer names the net of D1102.3 (I/O2), U1101.42 (UD-)
- net UDP: no longer names the net of D1102.1 (I/O1), U1101.43 (UD+)
- net XI: no longer names the net of C1101.1, U1101.5 (XI), Y1101.1
- net XO: no longer names the net of C1102.1, U1101.6 (XO), Y1101.2
Other:
- note removed: "Crystal, reset, TNOW strap pull-downs, ACT LED"
- note removed: "Test points (bring-up)"
- note removed: "USB 2.0 ESD (hub DS4 ↔ CH344 UD+/UD-)"
- moved on the sheet: C1101, C1102, C1103, C1104, C1105, C1106, C1107, C1108, D1101, D1102, R1101, R1102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
