File: backbone/usb-port.kicad_sch (KiCad schematic)
At the start: 0 parts

Commit message: before hand editing
Parts:
- added C801, C804: 100nF, 0_backbone:C_0603, symbol 0_backbone:C_0603
- added C802: 10uF, 0_backbone:C_0805, symbol 0_backbone:C_0805
- added C803: 47uF 10V, 0_backbone:C_1206, symbol 0_backbone:C_1206
- added C805, C806: 100nF, 0_backbone:C_0402, symbol 0_backbone:C_0402
- added C807: 1nF 2kV, 0_backbone:C_1206, symbol 0_backbone:C_1206
- added D801: USBLC6-2SC6, 0_backbone:SOT-23-6_L2.9-W1.6-P0.95-LS2.8-BL, symbol 0_backbone:USBLC6-2SC6_C2687116
- added D802: TPD4E05U06, 0_backbone:USON-10_L2.5-W1.0-P0.50-BL, symbol 0_backbone:TPD4E05U06DQAR_C138714
- added FB801: BLM21PG221SN1D, 0_backbone:FB_0805, symbol 0_backbone:FB_0805
- added J801: USB-A 3.0 receptacle, 0_backbone:USB-3.0-A-TH_HC-ST-003-01-Z, symbol 0_backbone:HC-ST-003-01-J
- added R801: 16.9k, 0_backbone:R_0603, symbol 0_backbone:R_0603
- added R802: 10k, 0_backbone:R_0603, symbol 0_backbone:R_0603
- added R803: 1M, 0_backbone:R_0603, symbol 0_backbone:R_0603
- added U801: TPS2553DBVR, 0_backbone:SOT-23-6_L2.9-W1.6-P0.95-LS2.8-BR, symbol 0_backbone:TPS2553DBVR
Connections:
- net DM: now also D801.4 (I/O2)
- net DP: now also D801.6 (I/O1)
- net OVERCUR_N: now also R802.2, U801.4 (/FAULT)
- net PWRCTL: now also U801.3 (EN)
- net SSRX_N: now also D802.5 (D2-), J801.5 (StdA_SSRX-)
- net SSRX_P: now also D802.4 (D2+), J801.6 (StdA_SSRX+)
- net SSTX_N: now also C806.1
- net SSTX_P: now also C805.1
- new net +3V3: R802.1
- new net +5V_USB: C801.1, C802.1, U801.1 (IN)
- new net DM_J: D801.3 (I/O2), J801.2 (D-)
- new net DP_J: D801.1 (I/O1), J801.3 (D+)
- new net GND: C801.2, C802.2, C803.2, C804.2, C807.2, D801.2 (GND), D802.3 (GND), D802.8 (GND), J801.4 (GND), J801.7 (GND_DRAIN), R801.2, R803.2, U801.2 (GND)
- new net ILIM: R801.1, U801.5 (ILIM)
- new net SHIELD: C807.1, J801.10 (SHELL), J801.11 (SHELL), R803.1
- new net SSTX_N_J: C806.2, D802.2 (D1-), J801.8 (StdA_SSTX-)
- new net SSTX_P_J: C805.2, D802.1 (D1+), J801.9 (StdA_SSTX+)
- new net VBUS_J: C804.1, D801.5 (VBUS), FB801.2, J801.1 (Vbus)
- new net VBUS_OUT: C803.1, FB801.1, U801.6 (OUT)
Other:
- note added: "ESD, AC coupling, receptacle"
- note added: "Net-class directives for the sheet-local nets"
- note added: "USB PORT — one sheet, instantiated 3× as usb-port-1..3 (hub DS1..DS3). Any device fits any port; identical 1.5 A limit on every port. Switch: TPS2553DBVR (replaces the SY6280 of the first draft: SY6280 has no fault output, so the hub's OVERCURxz could never see an over-current; TPS2553 FAULT is open-drain → OVERCUR_N, EN active high from PWRCTL). ILIM 16.9 k → 1.51 A nominal (IOS = 23950 / RILIM^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"
- note added: "VBUS switch (TPS2553, 1.5 A, fault → hub)"
- note removed: "USB PORT — one sheet, instantiated 3× as usb-port-1..3 (hub DS1..DS3). Any device fits any port. Golden reference: TUSB8041 EVM downstream port, datasheets/reference/ti-slvaf82b-esd-surge-protection-usb.pdf Parts (LCSC): SY6280AAC C55136 (Ilim = 6800 / Rset, 1.5 A on every port, EN must not float), TPD4E05U06 C138714, USBLC6-2 C2687116, USB-A 3.0 HC-ST-003-01-J C2845330 Pins: SSTX/SSRX (SSTX = hu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"
