File: backbone/usb-hub.kicad_sch (KiCad schematic)
At the start: 0 parts

Commit message: before hand editing
Parts:
- added C701, C715, C720: 10uF, 0_backbone:C_0805, symbol 0_backbone:C_0805
- added C702, C703: 30pF, 0_backbone:C_0603, symbol 0_backbone:C_0603
- added C704: 6.8pF, 0_backbone:C_0603, symbol 0_backbone:C_0603
- added C705: 4.7uF, 0_backbone:C_0805, symbol 0_backbone:C_0805
- added C706: 22uF, 0_backbone:C_0805, symbol 0_backbone:C_0805
- added C707, C708, C709, C710, C711, C712, C713, C714, C716, C717, C718, C719: 100nF, 0_backbone:C_0603, symbol 0_backbone:C_0603
- added FB701: BLM18PG221SN1D, 0_backbone:FB_0603, symbol 0_backbone:FB_0603
- added L701: 2.2uH 3.4A, 0_backbone:IND-SMD_L4.0-W4.0_LQH44PN2R2MP0L, symbol 0_backbone:SMNR4020-2.2UH
- added R701, R704, R705, R706, R707: 10k, 0_backbone:R_0603, symbol 0_backbone:R_0603
- added R702: 9.53k, 0_backbone:R_0603, symbol 0_backbone:R_0603
- added R703: 90.9k, 0_backbone:R_0603, symbol 0_backbone:R_0603
- added R708: 1M, 0_backbone:R_0603, symbol 0_backbone:R_0603
- added R709: 82k, 0_backbone:R_0603, symbol 0_backbone:R_0603
- added R710: 100k, 0_backbone:R_0603, symbol 0_backbone:R_0603
- added TP701: GRSTz, 0_backbone:TestPoint_Pad_D1.5mm, symbol 0_backbone:TestPoint
- added TP702: VDD_HUB, 0_backbone:TestPoint_Pad_D1.5mm, symbol 0_backbone:TestPoint
- added U701: TUSB8041IRGCR, 0_backbone:QFN-64_L9.0-W9.0-P0.50-BL-EP7.2, symbol 0_backbone:TUSB8041IRGCR
- added U702: TLV62569DBVR, 0_backbone:SOT-23-5_L3.0-W1.7-P0.95-LS2.8-BR, symbol 0_backbone:TLV62569DBVR
- added Y701: 24MHz 18pF, 0_backbone:OSC-SMD_4P-L3.2-W2.5-BL, symbol 0_backbone:Crystal_24MHz_3225
Connections:
- net +1V1_HUB: now also C704.1, C706.1, FB701.1, L701.2, R709.1
- net DS1_DM: now also U701.2 (USB_DM_DN1)
- net DS1_DP: now also U701.1 (USB_DP_DN1)
- net DS1_OVERCUR_N: now also R705.2, U701.46 (OVERCUR1z)
- net DS1_PWRCTL: now also U701.36 (PWRCTL1/BATEN1)
- net DS1_SSRX_N: now also U701.7 (USB_SSRXM_DN1)
- net DS1_SSRX_P: now also U701.6 (USB_SSRXP_DN1)
- net DS1_SSTX_N: now also U701.4 (USB_SSTXM_DN1)
- net DS1_SSTX_P: now also U701.3 (USB_SSTXP_DN1)
- net DS2_DM: now also U701.10 (USB_DM_DN2)
- net DS2_DP: now also U701.9 (USB_DP_DN2)
- net DS2_OVERCUR_N: now also R706.2, U701.47 (OVERCUR2z)
- net DS2_PWRCTL: now also U701.35 (PWRCTL2/BATEN2)
- net DS2_SSRX_N: now also U701.15 (USB_SSRXM_DN2)
- net DS2_SSRX_P: now also U701.14 (USB_SSRXP_DN2)
- net DS2_SSTX_N: now also U701.12 (USB_SSTXM_DN2)
- net DS2_SSTX_P: now also U701.11 (USB_SSTXP_DN2)
- net DS3_DM: now also U701.18 (USB_DM_DN3)
- net DS3_DP: now also U701.17 (USB_DP_DN3)
- net DS3_OVERCUR_N: now also R707.2, U701.44 (OVERCUR3z)
- net DS3_PWRCTL: now also U701.33 (PWRCTL3/BATEN3)
- net DS3_SSRX_N: now also U701.23 (USB_SSRXM_DN3)
- net DS3_SSRX_P: now also U701.22 (USB_SSRXP_DN3)
- net DS3_SSTX_N: now also U701.20 (USB_SSTXM_DN3)
- net DS3_SSTX_P: now also U701.19 (USB_SSTXP_DN3)
- net DS4_DM: now also U701.25 (USB_DM_DN4)
- net DS4_DP: now also U701.24 (USB_DP_DN4)
- net US_DM: now also U701.54 (USB_DM_UP)
- net US_DP: now also U701.53 (USB_DP_UP)
- net US_SSRX_N: now also U701.59 (USB_SSRXM_UP)
- net US_SSRX_P: now also U701.58 (USB_SSRXP_UP)
- net US_SSTX_N: now also U701.56 (USB_SSTXM_UP)
- net US_SSTX_P: now also U701.55 (USB_SSTXP_UP)
- new net +3V3: C716.1, C717.1, C718.1, C719.1, C720.1, R701.1, R705.1, R706.1, R707.1, U701.16 (VDD33), U701.34 (VDD33), U701.52 (VDD33), U701.63 (VDD33)
- new net +5V_USB: C705.1, U702.1 (EN), U702.4 (VIN)
- new net FB_1V1: C704.2, R709.2, R710.1, U702.5 (FB)
- new net GND: C701.2, C702.2, C703.2, C705.2, C706.2, C707.2, C708.2, C709.2, C710.2, C711.2, C712.2, C713.2, C714.2, C715.2, C716.2, C717.2, C718.2, C719.2, C720.2, R702.2, R704.2, R710.2, U701.49 (TEST), U701.65 (VSS), U702.2 (GND), Y701.2 (GND), Y701.4 (GND)
- new net GRSTz: C701.1, R701.2, TP701.1, U701.50 (GRSTz)
- new net SW_1V1: L701.1, U702.3 (SW)
- new net USB_R1: R702.1, U701.64 (USB_R1)
- new net USB_VBUS: R703.2, R704.1, U701.48 (USB_VBUS)
- new net VBUS: R703.1
- new net VDD_HUB: C707.1, C708.1, C709.1, C710.1, C711.1, C712.1, C713.1, C714.1, C715.1, FB701.2, TP702.1, U701.13 (VDD), U701.21 (VDD), U701.28 (VDD), U701.31 (VDD), U701.5 (VDD), U701.51 (VDD), U701.57 (VDD), U701.8 (VDD)
- new net XI: C702.1, R708.1, U701.62 (XI), Y701.1 (OSC)
- new net XO: C703.1, R708.2, U701.61 (XO), Y701.3 (OSC)
- no-connect marks 0 -> 13
Other:
- note added: "+1V1_HUB core: TLV62569, ferrite to VDD_HUB"
- note added: "24 MHz crystal"
- note added: "Reset, reference, VBUS sense, over-current pull-ups"
- note added: "USB HUB — TUSB8041 (4-port SS hub), 24 MHz crystal (18 pF CL, 2 × 30 pF, 1 MΩ feedback), 9.53 k on USB_R1, USB_VBUS = VBUS × 10 k / (90.9 k + 10 k). Straps (sampled at GRSTz release, all left at their internal defaults): FULLPWRMGMTz PD → power switching + over-current supported, GANGED PD → individual, PWRCTL_POL PU → PWRCTLx active high (TPS2553 EN), SMBUSz PU → I2C mode but no EEPROM fitted (D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"
- note added: "VDD_HUB (1.1 V core) and VDD33 decoupling"
- note removed: "USB HUB — TUSB8041 (4-port SS hub), 24 MHz crystal, 1.1 V core LDO, pin straps, GRSTz, USB_VBUS divider Golden reference: datasheets/reference/ti-sllu198-tusb8041-evm-users-guide.pdf (copy the EVM schematic), datasheets/tusb8041.pdf Parts (LCSC): TUSB8041IRGCR C544686 (D4: alternatives RTS5411S C5356838, CYUSB3304 C462531) Upstream: US_SSTX/SSRX + US_DP/DM from usbc-upstream. USB_VBUS sense from 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"

Commit message: schematics
Connections:
- net XI: now also C703.1, R708.2; no longer C702.1, R708.1
- net XO: now also C702.1, R708.1; no longer C703.1, R708.2
- net +1V1_HUB: no longer names the net of C704.1, C706.1, FB701.1, L701.2, R709.1
- net FB_1V1: no longer names the net of C704.2, R709.2, R710.1, U702.5 (FB)
- net GRSTz: no longer names the net of C701.1, R701.2, TP701.1, U701.50 (GRSTz)
- net SW_1V1: no longer names the net of L701.1, U702.3 (SW)
- net USB_R1: no longer names the net of R702.1, U701.64 (USB_R1)
- net USB_VBUS: no longer names the net of R703.2, R704.1, U701.48 (USB_VBUS)
Other:
- note removed: "24 MHz crystal"
- note removed: "Reset, reference, VBUS sense, over-current pull-ups"
- moved on the sheet: C701, C702, C703, C704, C705, C706, C707, C708, C709, C710, C711, C712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

Commit message: update
Connections:
- net XI: now also C702.1, R708.1; no longer C703.1, R708.2
- net XO: now also C703.1, R708.2; no longer C702.1, R708.1
- net GRSTz: now reaches C701.1, R701.2, TP701.1, U701.50 (GRSTz)
- net SW_1V1: now reaches L701.1, U702.3 (SW)
- net FB_1V1: now reaches C704.2, R709.2, R710.1, U702.5 (FB)
- net +1V1_HUB: now reaches C704.1, C706.1, FB701.1, L701.2, R709.1
- net USB_VBUS: now reaches R703.2, R704.1, U701.48 (USB_VBUS)
- net USB_R1: now reaches R702.1, U701.64 (USB_R1)
Other:
- note added: "24 MHz crystal"
- note added: "Reset, reference, VBUS sense, over-current pull-ups"
- moved on the sheet: C701, C702, C703, C704, C705, C706, C707, C708, C709, C710, C711, C712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
