File: backbone/usbc-upstream.kicad_sch (KiCad schematic)
At the start: 0 parts

Commit message: before hand editing
Parts:
- added C601, C602: 100nF, 0_backbone:C_0402, symbol 0_backbone:C_0402
- added C603, C604, C606: 100nF, 0_backbone:C_0603, symbol 0_backbone:C_0603
- added C605: 1uF, 0_backbone:C_0603, symbol 0_backbone:C_0603
- added C607: 1nF 2kV, 0_backbone:C_1206, symbol 0_backbone:C_1206
- added D601, D602: TPD4E05U06, 0_backbone:USON-10_L2.5-W1.0-P0.50-BL, symbol 0_backbone:TPD4E05U06DQAR_C138714
- added D603: USBLC6-2SC6, 0_backbone:SOT-23-6_L2.9-W1.6-P0.95-LS2.8-BL, symbol 0_backbone:USBLC6-2SC6_C2687116
- added J601: USB-C 24P receptacle, 0_backbone:USB-C-SMD_TYPE-C-24P-QT, symbol 0_backbone:TYPE-C24PQT
- added R601: 910k, 0_backbone:R_0603, symbol 0_backbone:R_0603
- added R602: 200k, 0_backbone:R_0603, symbol 0_backbone:R_0603
- added R603: 1M, 0_backbone:R_0603, symbol 0_backbone:R_0603
- added TP601: DIR, 0_backbone:TestPoint_Pad_D1.5mm, symbol 0_backbone:TestPoint
- added U601: HD3SS3220RNHR, 0_backbone:WQFN-30_L4.5-W2.5-P0.4-BL-EP, symbol 0_backbone:HD3SS3220RNHR
Connections:
- net US_DM: now also D603.4 (I/O2)
- net US_DP: now also D603.6 (I/O1)
- net US_SSRX_N: now also U601.10 (RXn)
- net US_SSRX_P: now also U601.9 (RXp)
- net US_SSTX_N: now also C602.1
- net US_SSTX_P: now also C601.1
- net VBUS: now also D603.5 (VBUS), J601.A4 (VBUS), J601.A9 (VBUS), J601.B4 (VBUS), J601.B9 (VBUS), R601.1
- new net +3V3: C603.1, C604.1, R602.1, U601.8 (VCC33)
- new net +5V_USB: C605.1, C606.1, U601.30 (VDD5)
- new net CC1: J601.A5 (CC1), U601.2 (CC1)
- new net CC2: J601.B5 (CC2), U601.1 (CC2)
- new net C_RX1N: D601.5 (D2-), J601.B10 (RX1-), U601.14 (RX1n)
- new net C_RX1P: D601.4 (D2+), J601.B11 (RX1+), U601.15 (RX1p)
- new net C_RX2N: D602.5 (D2-), J601.A10 (RX2-), U601.18 (RX2n)
- new net C_RX2P: D602.4 (D2+), J601.A11 (RX2+), U601.19 (RX2p)
- new net C_TX1N: D601.2 (D1-), J601.A3 (TX1-), U601.16 (TX1n)
- new net C_TX1P: D601.1 (D1+), J601.A2 (TX1+), U601.17 (TX1p)
- new net C_TX2N: D602.2 (D1-), J601.B3 (TX2-), U601.20 (TX2n)
- new net C_TX2P: D602.1 (D1+), J601.B2 (TX2+), U601.21 (TX2p)
- new net DIR: R602.2, TP601.1, U601.11 (DIR)
- new net DM_C: D603.3 (I/O2), J601.A7 (D-), J601.B7 (D-)
- new net DP_C: D603.1 (I/O1), J601.A6 (D+), J601.B6 (D+)
- new net GND: C603.2, C604.2, C605.2, C606.2, C607.2, D601.3 (GND), D601.8 (GND), D602.3 (GND), D602.8 (GND), D603.2 (GND), J601.A1 (GND), J601.A12 (GND), J601.B1 (GND), J601.B12 (GND), R603.2, U601.12 (ENn_MUX), U601.13 (GND), U601.28 (GND), U601.29 (ENn_CC), U601.3 (CURRENT_MODE), U601.31 (EP), U601.4 (PORT)
- new net SHIELD_C: C607.1, J601.25 (EP), J601.3 (EP), J601.4 (EP), R603.1
- new net SSTX_N_C: C602.2, U601.7 (TXn)
- new net SSTX_P_C: C601.2, U601.6 (TXp)
- new net VBUS_DET: R601.2, U601.5 (VBUS_DET)
- no-connect marks 0 -> 8
Other:
- note added: "AC coupling (hub SSTX) and straps"
- note added: "Decoupling (VCC33 2 × 100 nF, VDD5 1 µF + 100 nF)"
- note added: "ESD and the receptacle"
- note added: "Net-class directives for the sheet-local USB nets"
- note added: "USB-C UPSTREAM — J601 24-pin receptacle, HD3SS3220 in UFP / GPIO mode: PORT = GND (UFP), ADDR open (GPIO mode), ENn_CC = GND, ENn_MUX = GND, CURRENT_MODE = GND (don't care as UFP), VBUS_DET from the connector VBUS through 910 k, DIR pulled up 200 k (open drain, required). VBUS is detection only — never a power source; the VBUS net stays below 10 µF (kkh-analyze-schematic enforces it) and only fee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"
- note removed: "USB-C UPSTREAM — J3 receptacle, HD3SS3220 in UFP / GPIO mode, ESD Golden reference: datasheets/reference/ti-sllu241-hd3ss3220-ufp-dongle-evm.pdf, ti-slla481-hd3ss3220-schematic-checklist.pdf (run it before ERC) Parts (LCSC): HD3SS3220RNHR C165155, USB-C 24P receptacle C2681555 / C456013, TPD4E05U06 C138714 (SS), USBLC6-2 C2687116 (D+/D-) Straps: PORT = L (UFP), ADDR open (GPIO mode), ENn_CC = L, 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"

Commit message: schematics
Other:
- moved on the sheet: C603, C604, C605, C606, C607, D601, D602, D603, J601, R603

Commit message: update
Other:
- moved on the sheet: C603, C604, C605, C606, C607, D601, D602, D603, J601, R603
